File: hardware/Drone FCC/Barometro.kicad_sch (KiCad schematic)
At the start: 7 parts

Commit message: started schematic
Parts:
- U2: renamed from U?; footprint HLGA_10L_STM -> ILPS22QSTR:ILPS22QSTR
- gave numbers to parts that had none: 6
Changed lines of the file:
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@@
   (symbol (lib_id "power:GND") (at 193.04 82.55 0) (unit 1)
     (in_bom yes) (on_board yes) (fields_autoplaced)
-    (property "Reference" "#PWR?" (id 0) (at 193.04 88.9 0)
+    (property "Reference" "#PWR08" (id 0) (at 193.04 88.9 0)
       (effects (font (size 1.27 1.27)) hide)
     )
@@
   (symbol (lib_id "power:GND") (at 101.6 82.55 0) (unit 1)
     (in_bom yes) (on_board yes) (fields_autoplaced)
-    (property "Reference" "#PWR?" (id 0) (at 101.6 88.9 0)
+    (property "Reference" "#PWR06" (id 0) (at 101.6 88.9 0)
       (effects (font (size 1.27 1.27)) hide)
     )
@@
   (symbol (lib_id "Device:C_Small") (at 203.2 71.12 0) (unit 1)
     (in_bom yes) (on_board yes) (fields_autoplaced)
-    (property "Reference" "C?" (id 0) (at 205.74 69.8562 0)
+    (property "Reference" "C5" (id 0) (at 205.74 69.8562 0)
       (effects (font (size 1.27 1.27)) (justify left))
     )
@@
   (symbol (lib_id "power:GND") (at 175.26 82.55 0) (unit 1)
     (in_bom yes) (on_board yes) (fields_autoplaced)
-    (property "Reference" "#PWR?" (id 0) (at 175.26 88.9 0)
+    (property "Reference" "#PWR07" (id 0) (at 175.26 88.9 0)
       (effects (font (size 1.27 1.27)) hide)
     )
@@
   (symbol (lib_id "Device:R") (at 69.85 68.58 90) (unit 1)
     (in_bom yes) (on_board yes) (fields_autoplaced)
-    (property "Reference" "R?" (id 0) (at 69.85 62.2182 90))
+    (property "Reference" "R4" (id 0) (at 69.85 62.2182 90))
     (property "Value" "R" (id 1) (at 69.85 64.7582 90))
     (property "Footprint" "" (id 2) (at 69.85 70.358 90)
@@
   (symbol (lib_id "Device:C_Small") (at 193.04 71.12 0) (unit 1)
     (in_bom yes) (on_board yes) (fields_autoplaced)
-    (property "Reference" "C?" (id 0) (at 195.58 69.8562 0)
+    (property "Reference" "C4" (id 0) (at 195.58 69.8562 0)
       (effects (font (size 1.27 1.27)) (justify left))
     )
@@
   (symbol (lib_id "Device:R") (at 86.36 60.96 0) (unit 1)
     (in_bom yes) (on_board yes) (fields_autoplaced)
-    (property "Reference" "R?" (id 0) (at 88.9 59.6899 0)
+    (property "Reference" "R6" (id 0) (at 88.9 59.6899 0)
       (effects (font (size 1.27 1.27)) (justify left))
     )
@@
   (symbol (lib_id "Device:R") (at 77.47 60.96 0) (unit 1)
     (in_bom yes) (on_board yes) (fields_autoplaced)
-    (property "Reference" "R?" (id 0) (at 80.01 59.6899 0)
+    (property "Reference" "R5" (id 0) (at 80.01 59.6899 0)
       (effects (font (size 1.27 1.27)) (justify left))
     )
@@
   (symbol (lib_id "ILPS22QSTR:ILPS22QSTR") (at 107.95 66.04 0) (unit 1)
     (in_bom yes) (on_board yes) (fields_autoplaced)
-    (property "Reference" "U?" (id 0) (at 138.43 54.61 0)
+    (property "Reference" "U2" (id 0) (at 138.43 54.61 0)
       (effects (font (size 1.524 1.524)))
     )
@@
       (effects (font (size 1.524 1.524)))
     )
-    (property "Footprint" "HLGA_10L_STM" (id 2) (at 138.43 59.944 0)
+    (property "Footprint" "ILPS22QSTR:ILPS22QSTR" (id 2) (at 138.43 59.944 0)
       (effects (font (size 1.524 1.524)) hide)
     )
@@
   (symbol (lib_id "Device:R") (at 48.26 73.66 270) (mirror x) (unit 1)
     (in_bom yes) (on_board yes) (fields_autoplaced)
-    (property "Reference" "R?" (id 0) (at 48.26 67.31 90))
+    (property "Reference" "R3" (id 0) (at 48.26 67.31 90))
     (property "Value" "R" (id 1) (at 48.26 69.85 90))
     (property "Footprint" "" (id 2) (at 48.26 75.438 90)
