File: hardware/Drone FCC/modulo_GNSS.kicad_sch (KiCad schematic)
At the start: 2 parts

Commit message: started schematic
Parts:
- J1: renamed from J?; footprint (none) -> TSW-103-08-G-D-RA:SAMTEC_TSW-103-08-G-D-RA
- J2: renamed from J?; footprint (none) -> Connector_Hirose:Hirose_DF13C_CL535-0406-3-51_1x06-1MP_P1.25mm_Vertical
Changed lines of the file:
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@@
   (symbol (lib_id "power:GND") (at 86.36 80.01 0) (unit 1)
     (in_bom yes) (on_board yes) (fields_autoplaced)
-    (property "Reference" "#PWR?" (id 0) (at 86.36 86.36 0)
+    (property "Reference" "#PWR09" (id 0) (at 86.36 86.36 0)
       (effects (font (size 1.27 1.27)) hide)
     )
@@
   (symbol (lib_id "Connector_Generic:Conn_01x06") (at 85.09 60.96 0) (mirror y) (unit 1)
     (in_bom yes) (on_board yes) (fields_autoplaced)
-    (property "Reference" "J?" (id 0) (at 85.09 49.53 0))
+    (property "Reference" "J2" (id 0) (at 85.09 49.53 0))
     (property "Value" "GPS M8N" (id 1) (at 85.09 52.07 0))
-    (property "Footprint" "" (id 2) (at 85.09 60.96 0)
+    (property "Footprint" "Connector_Hirose:Hirose_DF13C_CL535-0406-3-51_1x06-1MP_P1.25mm_Vertical" (id 2) (at 85.09 60.96 0)
       (effects (font (size 1.27 1.27)) hide)
     )
@@
   (symbol (lib_id "Connector_Generic:Conn_02x03_Counter_Clockwise") (at 83.82 33.02 0) (unit 1)
     (in_bom yes) (on_board yes) (fields_autoplaced)
-    (property "Reference" "J?" (id 0) (at 85.09 24.13 0))
+    (property "Reference" "J1" (id 0) (at 85.09 24.13 0))
     (property "Value" "Conector GPS Auxiliar" (id 1) (at 85.09 26.67 0))
-    (property "Footprint" "" (id 2) (at 83.82 33.02 0)
+    (property "Footprint" "TSW-103-08-G-D-RA:SAMTEC_TSW-103-08-G-D-RA" (id 2) (at 83.82 33.02 0)
       (effects (font (size 1.27 1.27)) hide)
     )
