File: hardware/Drone FCC/sensores.kicad_sch (KiCad schematic)
At the start: 12 parts, among them J1 Mag Dupont, J19 GPS M8N - DF13, J2 GPS Dupont, J20 Mag DF13, U1 ICM-42688-V, U2 ILPS22QSTR

Commit message: add usb TVS diodes and mcu pin assignment
Changed lines of the file:
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@@
     (effects (font (size 1.27 1.27)) (justify right))
   )
-  (hierarchical_label "MAG_SDA" (shape input) (at 40.64 165.735 0)
+  (hierarchical_label "MAG_SDA" (shape bidirectional) (at 40.64 165.735 0)
     (effects (font (size 1.27 1.27)) (justify left))
   )

Commit message: rearranged FCC schematic
Changed lines of the file:
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@@
     (effects (font (size 1.27 1.27)) (justify right))
   )
-  (hierarchical_label "MAG_INT_DATA_RDY" (shape input) (at 40.64 160.655 0)
+  (hierarchical_label "MAG_INT_DATA_RDY" (shape output) (at 40.64 160.655 0)
     (effects (font (size 1.27 1.27)) (justify left))
   )
