File: hardware/Drone FCC/sensores.kicad_sch (KiCad schematic)
At the start: 12 parts, among them J201 Mag Dupont, J202 Mag DF13, J203 GPS Dupont, J204 GPS M8N - DF13, U201 ICM-42688-V, U202 ILPS22QSTR

Commit message: continued preliminar routing
Parts:
- C201: value 10n -> 10nF; footprint Capacitor_SMD:C_0603_1608Metric_Pad1.08x0.95mm_HandSolder -> Capacitor_SMD:C_0402_1005Metric_Pad0.74x0.62mm_HandSolder
- C202, C204, C205: value 0.1u -> 100nF; footprint Capacitor_SMD:C_0603_1608Metric_Pad1.08x0.95mm_HandSolder -> Capacitor_SMD:C_0402_1005Metric_Pad0.74x0.62mm_HandSolder
- C203: value 2.2u -> 2.2uF
Connections:
- net 3V3: no longer J202.1
- net 5V: now also J202.1, J204.1; no longer J204.6
- net GND: now also J204.6; no longer J204.1
- net GNSS_Rx: now also J204.3; no longer J204.4
- net GNSS_SCL: now also J204.4; no longer J204.3
- net GNSS_SDA: now also J204.5; no longer J204.2
- net GNSS_Tx: now also J204.2; no longer J204.5
Other:
- note removed: "¿HAY ALGÚN ORDENAMIENTO ESTÁNDAR PARA LOS PINES DE CADA CONECTOR?"
- moved on the sheet: J204
Changed lines of the file:
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@@
 (kicad_sch (version 20211123) (generator eeschema)
   (paper "A4")
-  (junction (at 140.335 187.325) (diameter 0) (color 0 0 0 0)
+  (junction (at 140.335 167.005) (diameter 0) (color 0 0 0 0)
   )
   (junction (at 100.965 50.165) (diameter 0) (color 0 0 0 0)
   )
   (junction (at 113.03 92.71) (diameter 0) (color 0 0 0 0)
+  )
+  (junction (at 140.335 169.545) (diameter 0) (color 0 0 0 0)
   )
   (junction (at 118.745 105.41) (diameter 0) (color 0 0 0 0)
@@
     (stroke (width 0) (type default) (color 0 0 0 0))
   )
+  (wire (pts (xy 140.335 169.545) (xy 163.83 169.545))
+    (stroke (width 0) (type default) (color 0 0 0 0))
+  )
   (polyline (pts (xy 107.95 138.43) (xy 107.95 196.85))
     (stroke (width 1) (type default) (color 0 0 0 0))
@@
     (stroke (width 0) (type default) (color 0 0 0 0))
   )
-  (wire (pts (xy 140.335 184.785) (xy 140.335 187.325))
+  (wire (pts (xy 140.335 164.465) (xy 140.335 167.005))
     (stroke (width 0) (type default) (color 0 0 0 0))
   )
@@
     (stroke (width 0) (type default) (color 0 0 0 0))
   )
-  (wire (pts (xy 137.16 184.785) (xy 140.335 184.785))
-    (stroke (width 0) (type default) (color 0 0 0 0))
-  )
-  (wire (pts (xy 137.16 187.325) (xy 140.335 187.325))
+  (wire (pts (xy 137.16 164.465) (xy 140.335 164.465))
+    (stroke (width 0) (type default) (color 0 0 0 0))
+  )
+  (wire (pts (xy 137.16 167.005) (xy 140.335 167.005))
     (stroke (width 0) (type default) (color 0 0 0 0))
   )
@@
     (stroke (width 0) (type default) (color 0 0 0 0))
   )
-  (wire (pts (xy 140.335 187.325) (xy 140.335 188.595))
+  (wire (pts (xy 140.335 167.005) (xy 140.335 169.545))
     (stroke (width 0) (type default) (color 0 0 0 0))
   )
@@
     (stroke (width 0) (type default) (color 0 0 0 0))
   )
-  (wire (pts (xy 137.16 169.545) (xy 163.83 169.545))
+  (wire (pts (xy 137.16 169.545) (xy 140.335 169.545))
     (stroke (width 0) (type default) (color 0 0 0 0))
   )
@@
     (effects (font (size 2.54 2.54)) (justify left bottom))
   )
-  (text "¿HAY ALGÚN ORDENAMIENTO\nESTÁNDAR PARA LOS PINES\nDE CADA CONECTOR?"
-    (at -48.895 173.355 0)
-    (effects (font (size 2.54 2.54) (thickness 0.254) bold) (justify left bottom))
-  )
   (label "GNSS_Rx" (at 149.225 177.165 180)
     (effects (font (size 1.27 1.27)) (justify right bottom))
@@
     )
   )
-  (global_label "3V3" (shape input) (at 95.25 168.91 0) (fields_autoplaced)
-    (effects (font (size 1.27 1.27)) (justify left))
-    (property "Intersheet References" "${INTERSHEET_REFS}" (id 0) (at 101.1707 168.8306 0)
+  (global_label "5V" (shape input) (at 95.25 168.91 0) (fields_autoplaced)
+    (effects (font (size 1.27 1.27)) (justify left))
+    (property "Intersheet References" "${INTERSHEET_REFS}" (id 0) (at 99.9612 168.8306 0)
       (effects (font (size 1.27 1.27)) (justify left) hide)
     )
@@
     (pin "1")
   )
-  (symbol (lib_id "DF13C-69-1.25v(51):DF13C-6P-1.25V(51)") (at 127 179.705 0) (mirror y) (unit 1)
+  (symbol (lib_id "DF13C-69-1.25v(51):DF13C-6P-1.25V(51)") (at 127 172.085 180) (unit 1)
     (in_bom yes) (on_board yes)
-    (property "Reference" "J204" (id 0) (at 127 160.655 0))
-    (property "Value" "GPS M8N - DF13" (id 1) (at 127 163.83 0))
-    (property "Footprint" "DF13C-6P-1.25V(51):HIROSE_DF13C-6P-1.25V(51)" (id 2) (at 127 179.705 0)
-      (effects (font (size 1.27 1.27)) (justify bottom) hide)
-    )
-    (property "Datasheet" "" (id 3) (at 127 179.705 0)
-      (effects (font (size 1.27 1.27)) hide)
-    )
-    (property "PARTREV" "N/A" (id 4) (at 127 179.705 0)
-      (effects (font (size 1.27 1.27)) (justify bottom) hide)
-    )
-    (property "STANDARD" "Manufacturer Recommendations" (id 5) (at 127 179.705 0)
-      (effects (font (size 1.27 1.27)) (justify bottom) hide)
-    )
-    (property "MAXIMUM_PACKAGE_HEIGHT" "5.1mm" (id 6) (at 127 179.705 0)
-      (effects (font (size 1.27 1.27)) (justify bottom) hide)
-    )
-    (property "MANUFACTURER" "Hirose Electric" (id 7) (at 127 179.705 0)
+    (property "Reference" "J204" (id 0) (at 127 191.135 0))
+    (property "Value" "GPS M8N - DF13" (id 1) (at 127 187.96 0))
+    (property "Footprint" "DF13C-6P-1.25V(51):HIROSE_DF13C-6P-1.25V(51)" (id 2) (at 127 172.085 0)
+      (effects (font (size 1.27 1.27)) (justify bottom) hide)
+    )
+    (property "Datasheet" "" (id 3) (at 127 172.085 0)
+      (effects (font (size 1.27 1.27)) hide)
+    )
+    (property "PARTREV" "N/A" (id 4) (at 127 172.085 0)
+      (effects (font (size 1.27 1.27)) (justify bottom) hide)
+    )
+    (property "STANDARD" "Manufacturer Recommendations" (id 5) (at 127 172.085 0)
+      (effects (font (size 1.27 1.27)) (justify bottom) hide)
+    )
+    (property "MAXIMUM_PACKAGE_HEIGHT" "5.1mm" (id 6) (at 127 172.085 0)
+      (effects (font (size 1.27 1.27)) (justify bottom) hide)
+    )
+    (property "MANUFACTURER" "Hirose Electric" (id 7) (at 127 172.085 0)
       (effects (font (size 1.27 1.27)) (justify bottom) hide)
     )
@@
       (effects (font (size 1.27 1.27)) (justify left))
     )
-    (property "Value" "2.2u" (id 1) (at 146.685 27.3112 0)
+    (property "Value" "2.2uF" (id 1) (at 146.685 27.3112 0)
       (effects (font (size 1.27 1.27)) (justify left))
     )
@@
       (effects (font (size 1.27 1.27)) (justify left))
     )
-    (property "Value" "0.1u" (id 1) (at 135.255 27.3112 0)
+    (property "Value" "100nF" (id 1) (at 135.255 27.3112 0)
       (effects (font (size 1.27 1.27)) (justify left))
     )
-    (property "Footprint" "Capacitor_SMD:C_0603_1608Metric_Pad1.08x0.95mm_HandSolder" (id 2) (at 132.715 26.035 0)
+    (property "Footprint" "Capacitor_SMD:C_0402_1005Metric_Pad0.74x0.62mm_HandSolder" (id 2) (at 132.715 26.035 0)
       (effects (font (size 1.27 1.27)) hide)
     )
@@
       (effects (font (size 1.27 1.27)) (justify right))
     )
-    (property "Value" "0.1u" (id 1) (at 24.13 83.8135 0)
+    (property "Value" "100nF" (id 1) (at 24.13 83.8135 0)
       (effects (font (size 1.27 1.27)) (justify right))
     )
-    (property "Footprint" "Capacitor_SMD:C_0603_1608Metric_Pad1.08x0.95mm_HandSolder" (id 2) (at 26.67 82.55 0)
+    (property "Footprint" "Capacitor_SMD:C_0402_1005Metric_Pad0.74x0.62mm_HandSolder" (id 2) (at 26.67 82.55 0)
       (effects (font (size 1.27 1.27)) hide)
     )
@@
       (effects (font (size 1.27 1.27)) (justify left))
     )
-    (property "Value" "10n" (id 1) (at 123.825 30.4862 0)
+    (property "Value" "10nF" (id 1) (at 123.825 30.4862 0)
       (effects (font (size 1.27 1.27)) (justify left))
     )
-    (property "Footprint" "Capacitor_SMD:C_0603_1608Metric_Pad1.08x0.95mm_HandSolder" (id 2) (at 121.285 29.21 0)
+    (property "Footprint" "Capacitor_SMD:C_0402_1005Metric_Pad0.74x0.62mm_HandSolder" (id 2) (at 121.285 29.21 0)
       (effects (font (size 1.27 1.27)) hide)
     )
@@
     (pin "1")
   )
-  (symbol (lib_id "power:GND") (at 140.335 188.595 0) (unit 1)
-    (in_bom yes) (on_board yes)
-    (property "Reference" "#PWR0175" (id 0) (at 140.335 194.945 0)
-      (effects (font (size 1.27 1.27)) hide)
-    )
-    (property "Value" "GND" (id 1) (at 140.335 193.675 0))
-    (property "Footprint" "" (id 2) (at 140.335 188.595 0)
-      (effects (font (size 1.27 1.27)) hide)
-    )
-    (property "Datasheet" "" (id 3) (at 140.335 188.595 0)
-      (effects (font (size 1.27 1.27)) hide)
-    )
-    (pin "1")
-  )
   (symbol (lib_id "power:GND") (at 100.965 53.975 0) (unit 1)
     (in_bom yes) (on_board yes) (fields_autoplaced)
@@
       (effects (font (size 1.27 1.27)) (justify left))
     )
-    (property "Value" "0.1u" (id 1) (at 121.92 99.0662 0)
+    (property "Value" "100nF" (id 1) (at 121.92 99.0662 0)
       (effects (font (size 1.27 1.27)) (justify left))
     )
-    (property "Footprint" "Capacitor_SMD:C_0603_1608Metric_Pad1.08x0.95mm_HandSolder" (id 2) (at 118.745 97.79 0)
-      (effects (font (size 1.27 1.27)) hide)
-    )
+    (property "Footprint" "Capacitor_SMD:C_0402_1005Metric_Pad0.74x0.62mm_HandSolder" (id 2) (at 118.745 97.79 0)
+      (effects (font (size 1.27 1.27)) hide)
+    )

Commit message: continue routing
Connections:
- net GND: now also J201.6 (Pin_6); no longer J201.2 (Pin_2)
- net MAG_INT_DATA_RDY: now also J201.5 (Pin_5); no longer J201.1 (Pin_1)
- net MAG_SCL: now also J201.2 (Pin_2); no longer J201.5 (Pin_5)
- net MAG_SDA: now also J201.1 (Pin_1); no longer J201.6 (Pin_6)
Changed lines of the file:
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@@
+    (stroke (width 0) (type default) (color 0 0 0 0))
+  )
+  (wire (pts (xy 23.495 186.69) (xy 32.385 186.69))
     (stroke (width 0) (type default) (color 0 0 0 0))
   )
@@
     (stroke (width 0) (type default) (color 0 0 0 0))
   )
-  (wire (pts (xy 23.495 191.77) (xy 32.385 191.77))
+  (wire (pts (xy 15.24 191.77) (xy 32.385 191.77))
     (stroke (width 0) (type default) (color 0 0 0 0))
   )
@@
     (stroke (width 1) (type default) (color 0 0 0 0))
   )
-  (wire (pts (xy 15.24 186.69) (xy 32.385 186.69))
-    (stroke (width 0) (type default) (color 0 0 0 0))
-  )
   (wire (pts (xy 95.885 42.545) (xy 100.965 42.545))
     (stroke (width 0) (type default) (color 0 0 0 0))
@@
     (stroke (width 0) (type default) (color 0 0 0 0))
   )
-  (wire (pts (xy 45.085 186.69) (xy 66.675 186.69))
-    (stroke (width 0) (type default) (color 0 0 0 0))
-  )
   (wire (pts (xy 95.885 22.225) (xy 121.285 22.225))
     (stroke (width 0) (type default) (color 0 0 0 0))
@@
     (stroke (width 0) (type default) (color 0 0 0 0))
   )
+  (wire (pts (xy 45.085 186.69) (xy 54.61 186.69))
+    (stroke (width 0) (type default) (color 0 0 0 0))
+  )
   (wire (pts (xy 45.085 189.23) (xy 55.88 189.23))
     (stroke (width 0) (type default) (color 0 0 0 0))
@@
     (stroke (width 0) (type default) (color 0 0 0 0))
   )
-  (wire (pts (xy 66.675 189.865) (xy 66.675 186.69))
+  (wire (pts (xy 54.61 194.945) (xy 54.61 191.77))
     (stroke (width 0) (type default) (color 0 0 0 0))
   )
@@
     (effects (font (size 1.27 1.27)) (justify right bottom))
   )
-  (label "MAG_SCL" (at 23.495 191.77 0)
-    (effects (font (size 1.27 1.27)) (justify left bottom))
+  (label "MAG_SCL" (at 54.61 186.69 180)
+    (effects (font (size 1.27 1.27)) (justify right bottom))
   )
   (label "GNSS_Rx" (at 175.895 154.305 0)
@@
     (effects (font (size 1.27 1.27)) (justify left bottom))
   )
-  (label "MAG_INT_DATA_RDY" (at 15.24 186.69 0)
+  (label "MAG_INT_DATA_RDY" (at 15.24 191.77 0)
     (effects (font (size 1.27 1.27)) (justify left bottom))
   )
@@
     (effects (font (size 1.27 1.27)) (justify right bottom))
   )
-  (label "MAG_SDA" (at 54.61 191.77 180)
-    (effects (font (size 1.27 1.27)) (justify right bottom))
+  (label "MAG_SDA" (at 23.495 186.69 0)
+    (effects (font (size 1.27 1.27)) (justify left bottom))
   )
   (label "GNSS_SDA" (at 149.225 172.085 180)
@@
     (pin "2")
   )
-  (symbol (lib_id "power:GND") (at 66.675 189.865 0) (unit 1)
-    (in_bom yes) (on_board yes) (fields_autoplaced)
-    (property "Reference" "#PWR0107" (id 0) (at 66.675 196.215 0)
-      (effects (font (size 1.27 1.27)) hide)
-    )
-    (property "Value" "GND" (id 1) (at 66.675 194.945 0))
-    (property "Footprint" "" (id 2) (at 66.675 189.865 0)
-      (effects (font (size 1.27 1.27)) hide)
-    )
-    (property "Datasheet" "" (id 3) (at 66.675 189.865 0)
-      (effects (font (size 1.27 1.27)) hide)
-    )
+  (symbol (lib_id "power:GND") (at 54.61 194.945 0) (unit 1)
+    (in_bom yes) (on_board yes) (fields_autoplaced)
+    (property "Reference" "#PWR0107" (id 0) (at 54.61 201.295 0)
+      (effects (font (size 1.27 1.27)) hide)
+    )
+    (property "Value" "GND" (id 1) (at 54.61 200.025 0))
+    (property "Footprint" "" (id 2) (at 54.61 194.945 0)
+      (effects (font (size 1.27 1.27)) hide)
+    )
+    (property "Datasheet" "" (id 3) (at 54.61 194.945 0)
+      (effects (font (size 1.27 1.27)) hide)
+    )

Commit message: routing: connected everything
Connections:
- net GND: now also J201.2 (Pin_2); no longer J201.6 (Pin_6)
- net MAG_INT_DATA_RDY: now also J201.1 (Pin_1); no longer J201.5 (Pin_5)
- net MAG_SCL: now also J201.5 (Pin_5); no longer J201.2 (Pin_2)
- net MAG_SDA: now also J201.6 (Pin_6); no longer J201.1 (Pin_1)
Changed lines of the file:
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@@
     (stroke (width 0) (type default) (color 0 0 0 0))
   )
-  (wire (pts (xy 23.495 186.69) (xy 32.385 186.69))
+  (wire (pts (xy 14.605 186.69) (xy 32.385 186.69))
     (stroke (width 0) (type default) (color 0 0 0 0))
   )
@@
   )
   (wire (pts (xy 140.335 164.465) (xy 140.335 167.005))
+    (stroke (width 0) (type default) (color 0 0 0 0))
+  )
+  (wire (pts (xy 64.77 186.69) (xy 64.77 191.135))
     (stroke (width 0) (type default) (color 0 0 0 0))
   )
@@
     (stroke (width 0) (type default) (color 0 0 0 0))
   )
-  (wire (pts (xy 45.085 186.69) (xy 54.61 186.69))
+  (wire (pts (xy 45.085 186.69) (xy 64.77 186.69))
     (stroke (width 0) (type default) (color 0 0 0 0))
   )
@@
   )
   (wire (pts (xy 95.885 29.845) (xy 100.33 29.845))
-    (stroke (width 0) (type default) (color 0 0 0 0))
-  )
-  (wire (pts (xy 54.61 194.945) (xy 54.61 191.77))
     (stroke (width 0) (type default) (color 0 0 0 0))
   )
@@
     (effects (font (size 1.27 1.27)) (justify right bottom))
   )
-  (label "MAG_SCL" (at 54.61 186.69 180)
-    (effects (font (size 1.27 1.27)) (justify right bottom))
+  (label "MAG_SCL" (at 15.24 191.77 0)
+    (effects (font (size 1.27 1.27)) (justify left bottom))
   )
   (label "GNSS_Rx" (at 175.895 154.305 0)
@@
     (effects (font (size 1.27 1.27)) (justify left bottom))
   )
-  (label "MAG_INT_DATA_RDY" (at 15.24 191.77 0)
+  (label "MAG_INT_DATA_RDY" (at 14.605 186.69 0)
     (effects (font (size 1.27 1.27)) (justify left bottom))
   )
@@
     (effects (font (size 1.27 1.27)) (justify right bottom))
   )
-  (label "MAG_SDA" (at 23.495 186.69 0)
-    (effects (font (size 1.27 1.27)) (justify left bottom))
+  (label "MAG_SDA" (at 54.61 191.77 180)
+    (effects (font (size 1.27 1.27)) (justify right bottom))
   )
   (label "GNSS_SDA" (at 149.225 172.085 180)
@@
     (pin "2")
   )
-  (symbol (lib_id "power:GND") (at 54.61 194.945 0) (unit 1)
-    (in_bom yes) (on_board yes) (fields_autoplaced)
-    (property "Reference" "#PWR0107" (id 0) (at 54.61 201.295 0)
-      (effects (font (size 1.27 1.27)) hide)
-    )
-    (property "Value" "GND" (id 1) (at 54.61 200.025 0))
-    (property "Footprint" "" (id 2) (at 54.61 194.945 0)
-      (effects (font (size 1.27 1.27)) hide)
-    )
-    (property "Datasheet" "" (id 3) (at 54.61 194.945 0)
-      (effects (font (size 1.27 1.27)) hide)
-    )
+  (symbol (lib_id "power:GND") (at 64.77 191.135 0) (unit 1)
+    (in_bom yes) (on_board yes) (fields_autoplaced)
+    (property "Reference" "#PWR0107" (id 0) (at 64.77 197.485 0)
+      (effects (font (size 1.27 1.27)) hide)
+    )
+    (property "Value" "GND" (id 1) (at 64.77 196.215 0))
+    (property "Footprint" "" (id 2) (at 64.77 191.135 0)
+      (effects (font (size 1.27 1.27)) hide)
+    )
+    (property "Datasheet" "" (id 3) (at 64.77 191.135 0)
+      (effects (font (size 1.27 1.27)) hide)
+    )
