File: hardware/Drone FCC/interfaz_can.kicad_sch (KiCad schematic)
At the start: 18 parts, among them J801 CAN 1 Connector 1, J802 CAN 1 Connector 2, J803 CAN 2 Connector 1, J804 CAN 2 Connector 2, U801 SN65HVD230, U802 SN65HVD230

Commit message: positioned components in 100x60 board with incomplete routing
Parts:
- removed J802: CAN 1 Connector 2, DF13A-3P-1.25H(21):HRS_DF13A-3P-1.25H(21), symbol DF13A-3P-1.25H(21):HRS_DF13A-3P-1.25H(21)
- removed J804: CAN 2 Connector 2, DF13A-3P-1.25H(21):HRS_DF13A-3P-1.25H(21), symbol DF13A-3P-1.25H(21):HRS_DF13A-3P-1.25H(21)
Connections:
- net CAN-: now reaches D801.1 (A1), J801.2, U801.6 (CANL)
- net CAN+: now reaches D801.2 (A2), J801.1, U801.7 (CANH)

Commit message: CAN PCB layout, positioned series resistors CAN TX and CAN RX
Parts:
- R801, R805: value 220 -> 51
- R802, R806: value 220 -> 510
Changed lines of the file:
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@@
     (in_bom yes) (on_board yes) (fields_autoplaced)
     (property "Reference" "R805" (id 0) (at 118.11 107.95 90))
-    (property "Value" "220" (id 1) (at 118.11 110.49 90))
+    (property "Value" "51" (id 1) (at 118.11 110.49 90))
     (property "Footprint" "Resistor_SMD:R_0402_1005Metric_Pad0.72x0.64mm_HandSolder" (id 2) (at 118.11 116.078 90)
       (effects (font (size 1.27 1.27)) hide)
@@
     (in_bom yes) (on_board yes) (fields_autoplaced)
     (property "Reference" "R802" (id 0) (at 107.95 45.72 90))
-    (property "Value" "220" (id 1) (at 107.95 48.26 90))
+    (property "Value" "510" (id 1) (at 107.95 48.26 90))
     (property "Footprint" "Resistor_SMD:R_0402_1005Metric_Pad0.72x0.64mm_HandSolder" (id 2) (at 107.95 53.848 90)
       (effects (font (size 1.27 1.27)) hide)
@@
     (in_bom yes) (on_board yes) (fields_autoplaced)
     (property "Reference" "R806" (id 0) (at 107.95 110.49 90))
-    (property "Value" "220" (id 1) (at 107.95 113.03 90))
+    (property "Value" "510" (id 1) (at 107.95 113.03 90))
     (property "Footprint" "Resistor_SMD:R_0402_1005Metric_Pad0.72x0.64mm_HandSolder" (id 2) (at 107.95 118.618 90)
       (effects (font (size 1.27 1.27)) hide)
@@
     (in_bom yes) (on_board yes) (fields_autoplaced)
     (property "Reference" "R801" (id 0) (at 118.11 43.18 90))
-    (property "Value" "220" (id 1) (at 118.11 45.72 90))
+    (property "Value" "51" (id 1) (at 118.11 45.72 90))
     (property "Footprint" "Resistor_SMD:R_0402_1005Metric_Pad0.72x0.64mm_HandSolder" (id 2) (at 118.11 51.308 90)
       (effects (font (size 1.27 1.27)) hide)

Commit message: continued routing missing connections
Connections:
- net GND: no longer J801.S1 (SHIELD), J801.S2 (SHIELD), J803.S1 (SHIELD), J803.S2 (SHIELD)
- no-connect marks 2 -> 6
Changed lines of the file:
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@@
   (junction (at 145.415 90.805) (diameter 0) (color 0 0 0 0)
   )
-  (junction (at 224.155 45.72) (diameter 0) (color 0 0 0 0)
-  )
   (junction (at 133.35 101.6) (diameter 0) (color 0 0 0 0)
   )
   (junction (at 133.35 90.805) (diameter 0) (color 0 0 0 0)
   )
-  (junction (at 224.155 113.03) (diameter 0) (color 0 0 0 0)
-  )
   (junction (at 145.415 26.035) (diameter 0) (color 0 0 0 0)
   )
-  (junction (at 224.155 48.26) (diameter 0) (color 0 0 0 0)
-  )
   (junction (at 173.355 116.84) (diameter 0) (color 0 0 0 0)
   )
@@
   (junction (at 133.35 26.035) (diameter 0) (color 0 0 0 0)
   )
-  (junction (at 224.155 110.49) (diameter 0) (color 0 0 0 0)
-  )
   (junction (at 133.35 36.83) (diameter 0) (color 0 0 0 0)
   )
+  (no_connect (at 226.06 45.72))
+  (no_connect (at 226.695 110.49))
+  (no_connect (at 226.06 48.26))
+  (no_connect (at 226.695 113.03))
   (no_connect (at 127 54.61))
   (no_connect (at 127 119.38))
-  (wire (pts (xy 224.155 113.03) (xy 224.155 116.205))
-    (stroke (width 0) (type default) (color 0 0 0 0))
-  )
-  (wire (pts (xy 224.155 113.03) (xy 227.965 113.03))
-    (stroke (width 0) (type default) (color 0 0 0 0))
-  )
-  (wire (pts (xy 224.155 43.18) (xy 224.155 45.72))
-    (stroke (width 0) (type default) (color 0 0 0 0))
-  )
   (wire (pts (xy 145.415 90.805) (xy 154.94 90.805))
     (stroke (width 0) (type default) (color 0 0 0 0))
@@
     (stroke (width 0) (type default) (color 0 0 0 0))
   )
+  (wire (pts (xy 226.695 113.03) (xy 227.965 113.03))
+    (stroke (width 0) (type default) (color 0 0 0 0))
+  )
   (wire (pts (xy 100.965 121.92) (xy 106.045 121.92))
     (stroke (width 0) (type default) (color 0 0 0 0))
@@
     (stroke (width 0) (type default) (color 0 0 0 0))
   )
+  (wire (pts (xy 226.06 45.72) (xy 227.965 45.72))
+    (stroke (width 0) (type default) (color 0 0 0 0))
+  )
   (wire (pts (xy 186.69 70.485) (xy 186.69 72.39))
     (stroke (width 0) (type default) (color 0 0 0 0))
@@
     (stroke (width 0) (type default) (color 0 0 0 0))
   )
-  (wire (pts (xy 224.155 48.26) (xy 224.155 51.435))
+  (wire (pts (xy 224.155 43.18) (xy 224.155 51.435))
     (stroke (width 0) (type default) (color 0 0 0 0))
   )
@@
     (stroke (width 0) (type default) (color 0 0 0 0))
   )
-  (wire (pts (xy 224.155 107.95) (xy 224.155 110.49))
-    (stroke (width 0) (type default) (color 0 0 0 0))
-  )
   (wire (pts (xy 113.665 121.92) (xy 135.255 121.92))
     (stroke (width 0) (type default) (color 0 0 0 0))
@@
     (stroke (width 0) (type default) (color 0 0 0 0))
   )
-  (wire (pts (xy 224.155 110.49) (xy 224.155 113.03))
+  (wire (pts (xy 224.155 107.95) (xy 224.155 116.205))
     (stroke (width 0) (type default) (color 0 0 0 0))
   )
@@
     (stroke (width 0) (type default) (color 0 0 0 0))
   )
-  (wire (pts (xy 224.155 45.72) (xy 224.155 48.26))
-    (stroke (width 0) (type default) (color 0 0 0 0))
-  )
   (wire (pts (xy 133.35 101.6) (xy 133.35 102.87))
     (stroke (width 0) (type default) (color 0 0 0 0))
   )
+  (wire (pts (xy 226.06 48.26) (xy 227.965 48.26))
+    (stroke (width 0) (type default) (color 0 0 0 0))
+  )
   (wire (pts (xy 100.965 116.84) (xy 104.14 116.84))
     (stroke (width 0) (type default) (color 0 0 0 0))
@@
     (stroke (width 0) (type default) (color 0 0 0 0))
   )
-  (wire (pts (xy 224.155 48.26) (xy 227.965 48.26))
-    (stroke (width 0) (type default) (color 0 0 0 0))
-  )
   (wire (pts (xy 118.745 26.035) (xy 118.745 29.21))
     (stroke (width 0) (type default) (color 0 0 0 0))
@@
     (stroke (width 0) (type default) (color 0 0 0 0))
   )
-  (wire (pts (xy 224.155 110.49) (xy 227.965 110.49))
-    (stroke (width 0) (type default) (color 0 0 0 0))
-  )
   (wire (pts (xy 133.35 99.06) (xy 133.35 101.6))
     (stroke (width 0) (type default) (color 0 0 0 0))
@@
     (stroke (width 0) (type default) (color 0 0 0 0))
   )
-  (wire (pts (xy 227.965 45.72) (xy 224.155 45.72))
-    (stroke (width 0) (type default) (color 0 0 0 0))
-  )
   (polyline (pts (xy 175.895 121.285) (xy 175.895 144.145))
     (stroke (width 0) (type default) (color 0 0 0 0))
@@
     (stroke (width 0) (type default) (color 0 0 0 0))
   )
+  (wire (pts (xy 226.695 110.49) (xy 227.965 110.49))
+    (stroke (width 0) (type default) (color 0 0 0 0))
+  )

Commit message: set values of resistors for LEDs
Other:
- moved on the sheet: J801, J803

Commit message: moved microSD to top layer. Also transistors for LEDs
Connections:
- net CAN+: now also J801.2; no longer J801.1
- net CAN-: now also J801.3; no longer J801.2
- net GND: now also J801.1, J803.1; no longer J801.3, J803.3
- net at D802.2 (A2), U802.7 (CANH): now also J803.2; no longer J803.1
- net at D802.1 (A1), U802.6 (CANL): now also J803.3; no longer J803.2
Other:
- moved on the sheet: J801, J803

Commit message: re routed CAN and USB with new dimensions
Connections:
- net CAN2+: now reaches D802.2 (A2), J803.2, U802.7 (CANH)
- net CAN2-: now reaches D802.1 (A1), J803.3, U802.6 (CANL)
- net CAN+ renamed CAN1+
- net CAN- renamed CAN1-
Changed lines of the file:
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@@
     (effects (font (size 1.27 1.27)) (justify left bottom))
   )
-  (label "CAN-" (at 187.325 54.61 0)
+  (label "CAN2+" (at 181.61 116.84 0)
     (effects (font (size 1.27 1.27)) (justify left bottom))
   )
-  (label "CAN+" (at 180.34 52.07 0)
+  (label "CAN2-" (at 188.595 119.38 0)
     (effects (font (size 1.27 1.27)) (justify left bottom))
   )
+  (label "CAN1-" (at 187.325 54.61 0)
+    (effects (font (size 1.27 1.27)) (justify left bottom))
+  )
+  (label "CAN1+" (at 180.34 52.07 0)
+    (effects (font (size 1.27 1.27)) (justify left bottom))
+  )
