File: hardware/Drone FCC/usb.kicad_sch (KiCad schematic)
At the start: 2 parts, among them J501 Micro USB - B, U501 USBLC6-2SC6

Commit message: continued preliminar routing
Connections:
- net USB_DM: now also U501.6 (I/O1); no longer J501.3 (D+), U501.3 (I/O2), U501.4 (I/O2)
- net USB_DP: now also U501.4 (I/O2); no longer J501.2 (D-), U501.1 (I/O1), U501.6 (I/O1)
- new net: J501.2 (D-), U501.1 (I/O1)
- new net: J501.3 (D+), U501.3 (I/O2)
Changed lines of the file:
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@@
   (junction (at 168.275 89.535) (diameter 0) (color 0 0 0 0)
-  )
-  (junction (at 133.35 104.775) (diameter 0) (color 0 0 0 0)
-  )
-  (junction (at 128.27 104.775) (diameter 0) (color 0 0 0 0)
-  )
-  (junction (at 133.35 73.66) (diameter 0) (color 0 0 0 0)
   )
   (junction (at 102.235 96.52) (diameter 0) (color 0 0 0 0)
   )
   (junction (at 102.235 99.06) (diameter 0) (color 0 0 0 0)
-  )
-  (junction (at 128.27 73.66) (diameter 0) (color 0 0 0 0)
   )
   (no_connect (at 99.568 91.44))
@@
     (stroke (width 0) (type default) (color 0 0 0 0))
   )
-  (wire (pts (xy 128.27 73.66) (xy 133.35 73.66))
-    (stroke (width 0) (type default) (color 0 0 0 0))
-  )
   (wire (pts (xy 133.35 73.66) (xy 156.21 73.66))
     (stroke (width 0) (type default) (color 0 0 0 0))
@@
     (stroke (width 0) (type default) (color 0 0 0 0))
   )
-  (wire (pts (xy 128.27 104.775) (xy 133.35 104.775))
-    (stroke (width 0) (type default) (color 0 0 0 0))
-  )
   (wire (pts (xy 133.35 73.66) (xy 133.35 79.375))
     (stroke (width 0) (type default) (color 0 0 0 0))
@@
     (effects (font (size 1.27 1.27)) (justify left bottom))
   )
-  (hierarchical_label "USB_DP" (shape bidirectional) (at 156.21 73.66 0)
+  (label "D-" (at 147.955 73.66 0)
+    (effects (font (size 1.27 1.27)) (justify left bottom))
+  )
+  (label "D+" (at 147.955 104.775 0)
+    (effects (font (size 1.27 1.27)) (justify left bottom))
+  )
+  (hierarchical_label "USB_DP" (shape bidirectional) (at 156.21 104.775 0)
     (effects (font (size 1.27 1.27)) (justify left))
   )
@@
     (effects (font (size 1.27 1.27)) (justify left))
   )
-  (hierarchical_label "USB_DM" (shape bidirectional) (at 156.21 104.775 0)
+  (hierarchical_label "USB_DM" (shape bidirectional) (at 156.21 73.66 0)
     (effects (font (size 1.27 1.27)) (justify left))
   )
