File: hardware/Drone FCC/usb.kicad_sch (KiCad schematic)
At the start: 2 parts, among them J501 Micro USB - B, U501 USBLC6-2SC6

Commit message: re enumeation of componentes
Parts:
- renumbered J501 to J25, U501 to U7
Changed lines of the file:
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@@
   (symbol (lib_id "power:GND") (at 115.57 93.345 0) (unit 1)
     (in_bom yes) (on_board yes) (fields_autoplaced)
-    (property "Reference" "#PWR0125" (id 0) (at 115.57 99.695 0)
+    (property "Reference" "#PWR059" (id 0) (at 115.57 99.695 0)
       (effects (font (size 1.27 1.27)) hide)
     )
@@
   (symbol (lib_name "105017-0001_1") (lib_id "105017-0001:105017-0001") (at 82.55 95.25 0) (unit 1)
     (in_bom yes) (on_board yes) (fields_autoplaced)
-    (property "Reference" "J501" (id 0) (at 82.55 76.2 0))
+    (property "Reference" "J25" (id 0) (at 82.55 76.2 0))
     (property "Value" "Micro USB - B" (id 1) (at 82.55 78.74 0))
     (property "Footprint" "105017-0001:MOLEX_105017-0001" (id 2) (at 82.55 110.49 0)
@@
   (symbol (lib_id "power:GND") (at 102.235 104.775 0) (mirror y) (unit 1)
     (in_bom yes) (on_board yes) (fields_autoplaced)
-    (property "Reference" "#PWR0126" (id 0) (at 102.235 111.125 0)
+    (property "Reference" "#PWR058" (id 0) (at 102.235 111.125 0)
       (effects (font (size 1.27 1.27)) hide)
     )
@@
   (symbol (lib_id "Power_Protection:USBLC6-2SC6") (at 130.81 89.535 270) (unit 1)
     (in_bom yes) (on_board yes)
-    (property "Reference" "U501" (id 0) (at 141.605 78.105 90))
+    (property "Reference" "U7" (id 0) (at 141.605 78.105 90))
     (property "Value" "USBLC6-2SC6" (id 1) (at 141.605 80.645 90))
     (property "Footprint" "Package_TO_SOT_SMD:SOT-23-6" (id 2) (at 118.11 89.535 0)
