File: hardware/Drone FCC/Drone FCC.kicad_pcb (KiCad board)
At the start: 4 copper layers, 308.8 x 80 mm, 211 parts, among them J1001 SPI externo, J1002 UART externa x2, J1003 I2C externo x2, J1004 UART externa x2, J1005 5V y 3V3 x 2, J201 Mag Dupont, J202 Mag DF13, J203 GPS Dupont, J204 GPS M8N - DF13, J301 ESC 1, J302 ESC 2, J303 ESC 3, J304 ESC 4, J305 ESC 5, J306 ESC 6, J307 ESC 7, J308 ESC 8, J309 SERVO 1, J310 SERVO 2, J311 SERVO 3, J312 SERVO 4, J313 Power Servo, J401 DSM Spektrum JST, J402 PPM Dupont, J501 Micro USB - B, J601 SWD Debug Connector, J701 DM3AT-SF-PEJM5, J801 CAN 1 Connector 1, J802 CAN 1 Connector 2, J803 CAN 2 Connector 1, J804 CAN 2 Connector 2, J901 PM02 PixHawk, Q1101 2N7002, Q1102 2N7002, Q1103 2N7002, Q1104 2N7002, Q1105 2N7002, Q1106 2N7002, Q1107 2N7002, Q1108 2N7002, Q901 Q_PMOS_GSD, SW101 SW RESET, SW1101 SW Propósito General, SW1102 SW Propósito General, U101 STM32F746ZGTx, U201 ICM-42688-V, U202 ILPS22QSTR, U501 USBLC6-2SC6, U801 SN65HVD230, U802 SN65HVD230, U901 ZLDO1117QG33TA, Y101 12MHz, Y102 32.768kHz

Commit message: continued preliminar routing
Parts:
- removed C803, C806: 100nF, Capacitor_SMD:C_0402_1005Metric_Pad0.74x0.62mm_HandSolder
- removed the D903 at (237.3, 106.3)
- removed the D903 at (446.1, 91.2)
- removed the J1001 at (384.6, 132.7)
- removed the J1002 at (384.6, 112.4)
- removed the J1003 at (398.0, 154.7)
- removed the J1003 at (213.9, 149.4)
- removed the J1004 at (384.6, 122.5)
- removed the J1005 at (433.2, 89.1)
- removed the J201 at (450.3, 137.9)
- removed the J202 at (453.1, 151.1)
- removed the J203 at (450.3, 130.3)
- removed the J204 at (454.1, 120.5)
- removed the J301 at (426.1, 160.2)
- removed the J302 at (428.7, 160.2)
- removed the J303 at (431.2, 160.2)
- removed the J304 at (433.7, 160.2)
- removed the J305 at (436.3, 160.2)
- removed the J306 at (438.8, 160.2)
- removed the J307 at (441.4, 160.2)
- removed the J308 at (443.9, 160.2)
- removed the J309 at (400.6, 160.2)
- removed the J310 at (403.1, 160.2)
- removed the J311 at (405.7, 160.2)
- removed the J312 at (408.2, 160.2)
- removed the J313 at (159.5, 116.7)
- removed the J313 at (414.4, 151.2)
- removed the J401 at (379.7, 140.6)
- removed the J402 at (382.0, 153.2)
- removed the J501 at (454.5, 108.7)
- removed the J601 at (486.6, 105.8)
- removed the J701 at (417.8, 99.5)
- removed the J801 at (390.5, 85.6)
- removed the J801 at (168.3, 100.3)
- removed the J802 at (400.3, 85.5)
- removed the J802 at (178.4, 100.3)
- removed the J803 at (400.7, 85.8)
- removed the J804 at (390.8, 85.9)
- removed the J901 at (245.7, 109.9)
- removed the J901 at (454.4, 95.3)
- removed R101, R102: R, Resistor_SMD:R_0402_1005Metric_Pad0.72x0.64mm_HandSolder
- removed R804, R808: 5.1k, Resistor_SMD:R_0402_1005Metric_Pad0.72x0.64mm_HandSolder
- removed the U101 at (436.1, 110.9)
- removed the U201 at (417.3, 121.7)
- removed the U501 at (447.5, 109.1)
- removed the U801 at (174.5, 110.1)
- removed the U801 at (392.0, 95.4)
- removed the U802 at (395.2, 95.2)
- removed the U901 at (258.6, 98.9)
- removed the U901 at (434.1, 96.6)
- added C1: 100nF, Capacitor_SMD:C_0603_1608Metric_Pad1.08x0.95mm_HandSolder, F.Cu at (108.1, 74.2)
- added C2: 100nF, Capacitor_SMD:C_0603_1608Metric_Pad1.08x0.95mm_HandSolder, F.Cu at (187.6, 74.2)
- added C3: 100nF, Capacitor_SMD:C_0603_1608Metric_Pad1.08x0.95mm_HandSolder, F.Cu at (187.5, 145.4)
- added C4: 100nF, Capacitor_SMD:C_0603_1608Metric_Pad1.08x0.95mm_HandSolder, F.Cu at (108.4, 145.4)
- added D903: PMEG60T30ELRX, PMEG60T30ELRX:SODFL3517X110N, F.Cu at (176.8, 78.8)
- added H1: MountingHole_Pad, MountingHole:MountingHole_3.2mm_M3_Pad_TopBottom, F.Cu at (102.4, 74.2)
- added H2: MountingHole_Pad, MountingHole:MountingHole_3.2mm_M3_Pad_TopBottom, F.Cu at (193.3, 74.2)
- added H3: MountingHole_Pad, MountingHole:MountingHole_3.2mm_M3_Pad_TopBottom, F.Cu at (193.2, 145.4)
- added H4: MountingHole_Pad, MountingHole:MountingHole_3.2mm_M3_Pad_TopBottom, F.Cu at (102.4, 145.4)
- added J1003: I2C externo x2, Connector_PinHeader_2.54mm:PinHeader_2x05_P2.54mm_Horizontal, F.Cu at (190.5, 100.1)
- added J313: Power Servo, 1935161:PHOENIX_1935161, F.Cu at (117.7, 144.8)
- added J801: CAN 1 Connector 1, DF13A-3P-1.25H(21):HRS_DF13A-3P-1.25H(21), F.Cu at (101.2, 83.1)
- added J802: CAN 1 Connector 2, DF13A-3P-1.25H(21):HRS_DF13A-3P-1.25H(21), B.Cu at (101.2, 83.1)
- added J901: PM02 PixHawk, DF13C-6P-1.25V(51):HIROSE_DF13C-6P-1.25V(51), F.Cu at (177.3, 72.3)
- added U801: SN65HVD230, Package_SO:SOIC-8_3.9x4.9mm_P1.27mm, F.Cu at (116.9, 83.6)
- added U901: ZLDO1117QG33TA, Package_TO_SOT_SMD:SOT-223-3_TabPin2, F.Cu at (167.1, 85.1)
- C101, C102, C104, C105, C106, C107, C108, C109, C110, C111, C112, C113, C114, C115, C802: footprint Capacitor_SMD:C_0603_1608Metric_Pad1.08x0.95mm_HandSolder -> Capacitor_SMD:C_0402_1005Metric_Pad0.74x0.62mm_HandSolder
- C116: footprint Capacitor_SMD:C_0805_2012Metric_Pad1.18x1.45mm_HandSolder -> Capacitor_SMD:C_0603_1608Metric_Pad1.08x0.95mm_HandSolder
- C117, C118: footprint Capacitor_SMD:C_1206_3216Metric_Pad1.33x1.80mm_HandSolder -> Capacitor_SMD:C_0603_1608Metric_Pad1.08x0.95mm_HandSolder
- C201: value 10n -> 10nF; footprint Capacitor_SMD:C_0603_1608Metric_Pad1.08x0.95mm_HandSolder -> Capacitor_SMD:C_0402_1005Metric_Pad0.74x0.62mm_HandSolder
- C202, C204, C205: value 0.1u -> 100nF; footprint Capacitor_SMD:C_0603_1608Metric_Pad1.08x0.95mm_HandSolder -> Capacitor_SMD:C_0402_1005Metric_Pad0.74x0.62mm_HandSolder
- C203: value 2.2u -> 2.2uF
- C804, R702, R703, R704, R705, R706, R805, R806, R807: moved to B.Cu
- C805: footprint Capacitor_SMD:C_0603_1608Metric_Pad1.08x0.95mm_HandSolder -> Capacitor_SMD:C_0402_1005Metric_Pad0.74x0.62mm_HandSolder; moved to B.Cu
- J701, J803: moved to F.Cu
- moved C116 427.8 mm to (349.5, 96.8)
- moved U202 261.0 mm to (153.7, 116.7), turned to 180 degrees
- moved C119 243.9 mm to (126.5, 31.0)
- moved R104 243.4 mm to (173.3, 118.8), turned to -45 degrees
- moved SW101 242.2 mm to (114.8, 29.5)
- moved R112 242.0 mm to (157.9, 89.2), turned to 90 degrees
- moved R111 237.3 mm to (156.1, 89.2), turned to -90 degrees
- moved D802 236.9 mm to (109.8, 92.5), turned to 0 degrees
- moved C117 234.4 mm to (143.5, 113.7), turned to -45 degrees
- moved D801 233.1 mm to (109.8, 83.6)
- moved R103 229.7 mm to (172.3, 119.8), turned to -45 degrees
- moved R105 223.3 mm to (146.6, 116.4), turned to -90 degrees
- moved C124 219.2 mm to (136.2, 98.4), turned to -45 degrees
- moved R106 214.7 mm to (149.9, 119.0), turned to 90 degrees
- moved C113 213.8 mm to (138.6, 117.0), turned to -135 degrees
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Connections:
- net Net-(C903-Pad1) renamed /Alimentación/5Vin
- D902 pad 2: Net-(D902-Pad2) -> /Vbus
- J1001 pad 1: /Conexiones_extra/SPI_SCK -> 5V
- J1001 pad 6: GND -> /Conexiones_extra/SPI_SCK
- J1001 pad 8: 5V -> GND
- J202 pad 1: 3V3 -> 5V
- J204 pad 1: GND -> 5V
- J204 pad 2: /Sensores/GNSS_SDA -> /Sensores/GNSS_Tx
- J204 pad 3: /Sensores/GNSS_SCL -> /Sensores/GNSS_Rx
- J204 pad 4: /Sensores/GNSS_Rx -> /Sensores/GNSS_SCL
- J204 pad 5: /Sensores/GNSS_Tx -> /Sensores/GNSS_SDA
- J204 pad 6: 5V -> GND
- J305 pad 1: /MCU/TIM4_CH1 -> /MCU/TIM1_CH1
- J306 pad 1: /MCU/TIM4_CH2 -> /MCU/TIM1_CH2
- J307 pad 1: /MCU/TIM4_CH3 -> /MCU/TIM1_CH3
- J308 pad 1: /MCU/TIM4_CH4 -> /MCU/TIM1_CH4
- J309 pad 1: /MCU/TIM1_CH1 -> /MCU/TIM2_CH1
- J310 pad 1: /MCU/TIM1_CH2 -> /MCU/TIM2_CH2
- J311 pad 1: /MCU/TIM1_CH3 -> /MCU/TIM2_CH3
- J312 pad 1: /MCU/TIM1_CH4 -> /MCU/TIM2_CH4
- J402 pad 3: /MCU/TIM2_CH3 -> /RC control/PPM
- J501 pad 2: /MCU/OTG_FS_DP -> Net-(J501-Pad2)
- J501 pad 3: /MCU/OTG_FS_DM -> Net-(J501-Pad3)
- J803 pad 1: Net-(D802-Pad1) -> Net-(D802-Pad2)
- J803 pad 2: Net-(D802-Pad2) -> Net-(D802-Pad1)
- J804 pad 1: Net-(D802-Pad1) -> Net-(D802-Pad2)
- J804 pad 2: Net-(D802-Pad2) -> Net-(D802-Pad1)
- Q901 pad 3: Net-(D902-Pad2) -> Net-(Q901-Pad3)
- R807 pad 2: Net-(C806-Pad2) -> Net-(R807-Pad2)
- R901 pad 1: Net-(D902-Pad2) -> Net-(Q901-Pad3)
- U101 pad 1: /Conexiones_extra/SPI_SCK -> unconnected-(U101-Pad1)
- U101 pad 103: /MCU/OTG_FS_DM -> /USB/D-
- U101 pad 104: /MCU/OTG_FS_DP -> /USB/D+
- U101 pad 15: /MCU/PF_5(EXTI5) -> /Conexiones_extra/SPI_EOC
- U101 pad 18: /MCU/SPI5_CS -> /Conexiones_extra/SPI_CS
- U101 pad 19: /MCU/SPI5_SCK -> /Conexiones_extra/SPI_SCK
- U101 pad 2: /Conexiones_extra/SPI_EOC -> /MCU/PE_3(EXTI3)
- U101 pad 20: /MCU/SPI5_MISO -> /Conexiones_extra/SPI_MISO
- U101 pad 21: /MCU/SPI5_MOSI -> /Conexiones_extra/SPI_MOSI
- U101 pad 3: /Conexiones_extra/SPI_CS -> unconnected-(U101-Pad3)
- U101 pad 34: /Conexiones_extra/UARTC_TX -> /MCU/TIM2_CH1
- U101 pad 35: /Conexiones_extra/UARTC_RX -> /MCU/TIM2_CH2
- U101 pad 37: unconnected-(U101-Pad37) -> /MCU/TIM2_CH4
- U101 pad 4: /Conexiones_extra/SPI_MISO -> unconnected-(U101-Pad4)
- U101 pad 5: /Conexiones_extra/SPI_MOSI -> unconnected-(U101-Pad5)
- U101 pad 73: unconnected-(U101-Pad73) -> /MCU/SPI2_CS
- U101 pad 74: unconnected-(U101-Pad74) -> /MCU/SPI2_SCK
- U101 pad 75: unconnected-(U101-Pad75) -> /MCU/SPI2_MISO
- U101 pad 76: unconnected-(U101-Pad76) -> /MCU/SPI2_MOSI
- U201 pad 1: /MCU/SPI5_MISO -> /MCU/SPI2_MISO
- U201 pad 12: /MCU/SPI5_CS -> /MCU/SPI2_CS
- U201 pad 13: /MCU/SPI5_SCK -> /MCU/SPI2_SCK
- U201 pad 14: /MCU/SPI5_MOSI -> /MCU/SPI2_MOSI
- U201 pad 4: /MCU/PF_5(EXTI5) -> /MCU/PE_3(EXTI3)
- U501 pad 1: /MCU/OTG_FS_DP -> Net-(J501-Pad2)
- U501 pad 3: /MCU/OTG_FS_DM -> Net-(J501-Pad3)
- U501 pad 4: /MCU/OTG_FS_DM -> /USB/D+
- U501 pad 6: /MCU/OTG_FS_DP -> /USB/D-
- U802 pad 6: Net-(D802-Pad2) -> Net-(D802-Pad1)
- U802 pad 7: Net-(D802-Pad1) -> Net-(D802-Pad2)
- U802 pad 8: Net-(R808-Pad2) -> Net-(R807-Pad2)
Routing:
- net 5V: track 0.00 -> 95.1 mm
- net GND: track 11.4 -> 92.2 mm, vias 1 -> 12
- net 3V3: track 7.50 -> 82.7 mm
- net /MCU/TIM1_CH4: track 0.00 -> 35.7 mm
- net /MCU/TIM1_CH3: track 0.00 -> 34.5 mm
- net /USB/D-: track 0.00 -> 34.1 mm
- net /USB/D+: track 0.00 -> 33.6 mm
- net /MCU/TIM1_CH2: track 0.00 -> 33.4 mm
- net /MCU/TIM1_CH1: track 0.00 -> 31.2 mm
- net /Sensores/GNSS_SCL: track 0.00 -> 27.5 mm, vias 0 -> 4
- net /MCU/TIM3_CH4: track 0.00 -> 27.3 mm
- net /MCU/TIM3_CH3: track 0.00 -> 26.1 mm
- net Net-(R802-Pad2): track 0.00 -> 25.1 mm
- net /MCU/PF_5(EXTI5): track 25.0 -> 0.00 mm
- net /MCU/TIM3_CH2: track 0.00 -> 24.8 mm
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- added copper zone on In2.Cu, net 3V3
- added copper zone on In1.Cu, net GND
Other:
- board size 308.8 x 80 mm -> 100 x 80 mm

Commit message: continue routing
Parts:
- moved J201 45.8 mm to (190.5, 100.2), turned to 0 degrees
- moved R103 28.0 mm to (149.8, 103.2)
- moved R104 27.4 mm to (152.1, 101.4)
- moved J1002 21.1 mm to (173.0, 142.6), turned to -90 degrees
- moved J401 18.0 mm to (158.2, 98.9)
- moved J1001 17.8 mm to (190.4, 130.7)
- moved C4 8.40 mm to (102.4, 139.4), turned to 90 degrees
- moved J1003 7.69 mm to (190.6, 107.8)
- moved J202 6.41 mm to (171.4, 110.0)
- moved J204 6.41 mm to (170.2, 96.8)
- turned H4 to 90 degrees
Connections:
- J1001 pad 2: /Conexiones_extra/SPI_MOSI -> /Conexiones_extra/SPI_EOC
- J1001 pad 3: /Conexiones_extra/SPI_CS -> /Conexiones_extra/SPI_SCK
- J1001 pad 4: /Conexiones_extra/SPI_MISO -> /Conexiones_extra/SPI_CS
- J1001 pad 5: /Conexiones_extra/SPI_EOC -> /Conexiones_extra/SPI_MOSI
- J1001 pad 6: /Conexiones_extra/SPI_SCK -> /Conexiones_extra/SPI_MISO
- J1003 pad 1: 5V -> /Conexiones_extra/I2CA_SDA
- J1003 pad 10: /Conexiones_extra/I2CA_SDA -> /Conexiones_extra/I2CA_SCL
- J1003 pad 2: /Conexiones_extra/I2CA_SCL -> /Conexiones_extra/I2CA_SDA
- J1003 pad 4: /Conexiones_extra/I2CA_SDA -> 3V3
- J1003 pad 7: 3V3 -> 5V
- J1003 pad 8: /Conexiones_extra/I2CA_SCL -> 3V3
- J1003 pad 9: 3V3 -> /Conexiones_extra/I2CA_SCL
- J201 pad 1: /Sensores/MAG_INT_DATA_RDY -> /Sensores/GNSS_SDA
- J201 pad 2: GND -> /Sensores/GNSS_SCL
- J201 pad 5: /Sensores/GNSS_SCL -> /Sensores/MAG_INT_DATA_RDY
- J201 pad 6: /Sensores/GNSS_SDA -> GND
- J401 pad 3: /MCU/UART7_RX -> /MCU/USART3_RX
- J402 pad 3: /RC control/PPM -> /MCU/TIM4_CH1
- U101 pad 119: /Conexiones_extra/UARTB_TX -> /Sensores/GNSS_Tx
- U101 pad 122: /Conexiones_extra/UARTB_RX -> /Sensores/GNSS_Rx
- U101 pad 77: /Sensores/GNSS_Tx -> /MCU/USART3_TX
- U101 pad 78: /Sensores/GNSS_Rx -> /MCU/USART3_RX
Routing:
- net /Conexiones_extra/SPI_EOC: track 0.00 -> 86.4 mm, vias 0 -> 1
- net /Conexiones_extra/SPI_CS: track 0.00 -> 86.2 mm, vias 0 -> 1
- net /Conexiones_extra/SPI_MISO: track 0.00 -> 86.1 mm, vias 0 -> 1
- net /MCU/TIM4_CH1: track 0.00 -> 85.2 mm, vias 0 -> 1
- net /Conexiones_extra/SPI_SCK: track 0.00 -> 82.9 mm, vias 0 -> 1
- net /Conexiones_extra/SPI_MOSI: track 0.00 -> 81.7 mm, vias 0 -> 1
- net /Conexiones_extra/I2CA_SDA: track 0.00 -> 75.7 mm, vias 0 -> 1
- net /Sensores/GNSS_Rx: track 15.3 -> 84.8 mm, vias 1 -> 2
- net /Conexiones_extra/I2CA_SCL: track 0.00 -> 69.2 mm, vias 0 -> 1
- net /Sensores/GNSS_Tx: track 12.2 -> 80.4 mm, vias 1 -> 2
- net /Sensores/MAG_INT_DATA_RDY: track 0.00 -> 66.5 mm, vias 0 -> 1
- net /Sensores/GNSS_SCL: track 27.5 -> 92.2 mm
- net /Sensores/GNSS_SDA: track 23.4 -> 83.9 mm, vias 2 -> 3
- net /MCU/USART3_RX: track 0.00 -> 33.3 mm, vias 0 -> 2
- net 5V: track 95.1 -> 121.6 mm
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
Commit message: routing: connected everything
Parts:
- removed C1, C2, C3, C4: 100nF, Capacitor_SMD:C_0603_1608Metric_Pad1.08x0.95mm_HandSolder
- removed J1002, J1004: UART externa x2, Connector_PinHeader_2.54mm:PinHeader_2x04_P2.54mm_Horizontal
- added J1: Conn_02x06_Odd_Even, Connector_PinHeader_2.54mm:PinHeader_2x06_P2.54mm_Horizontal, F.Cu at (172.1, 77.1)
- C804, C805, D802, R705, R706, R805, R806, R807, U802: moved to F.Cu
- moved R907 146.1 mm to (115.2, 124.6), turned to 90 degrees
- moved R906 144.4 mm to (113.9, 124.6), turned to 90 degrees
- moved J901 75.2 mm to (176.1, 147.5), turned to 0 degrees
- moved D903 60.2 mm to (171.7, 138.8), turned to -90 degrees
- moved J804 58.1 mm to (68.0, 45.5)
- moved C905 52.5 mm to (167.2, 138.3), turned to 180 degrees
- moved C904 50.4 mm to (167.4, 135.7), turned to 180 degrees
- moved C903 49.0 mm to (175.6, 131.8), turned to 90 degrees
- moved J1005 47.9 mm to (190.4, 130.3)
- moved U901 44.4 mm to (169.3, 129.4), turned to 90 degrees
- moved R701 42.0 mm to (78.1, 100.6), turned to 90 degrees
- moved C108 35.8 mm to (83.3, 97.4), turned to 0 degrees
- moved C109 35.5 mm to (82.4, 89.8), turned to 0 degrees
- moved J802 35.4 mm to (81.9, 53.3)
- moved R108 28.7 mm to (83.9, 93.9), turned to 90 degrees
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Connections:
- C903 pad 1: /Alimentación/5Vin -> 5V
- D902 pad 1: /Alimentación/5Vin -> 5V
- D903 pad 1: /Alimentación/5Vin -> 5V
- D903 pad 2: 5V -> /Alimentación/5Vin
- H1 pad 1: Net-(C1-Pad1) -> GND
- H2 pad 1: Net-(C2-Pad1) -> GND
- H3 pad 1: Net-(C3-Pad1) -> GND
- H4 pad 1: Net-(C4-Pad1) -> GND
- J1003 pad 1: /Conexiones_extra/I2CA_SDA -> /Conexiones_extra/I2CA_SCL
- J1003 pad 10: /Conexiones_extra/I2CA_SCL -> /Conexiones_extra/I2CA_SDA
- J1003 pad 2: /Conexiones_extra/I2CA_SDA -> /Conexiones_extra/I2CA_SCL
- J1003 pad 9: /Conexiones_extra/I2CA_SCL -> /Conexiones_extra/I2CA_SDA
- J201 pad 1: /Sensores/GNSS_SDA -> /Sensores/MAG_INT_DATA_RDY
- J201 pad 2: /Sensores/GNSS_SCL -> GND
- J201 pad 5: /Sensores/MAG_INT_DATA_RDY -> /Sensores/GNSS_SCL
- J201 pad 6: GND -> /Sensores/GNSS_SDA
- J401 pad 3: /MCU/USART3_RX -> /MCU/UART7_RX
- J901 pad 1: 5V -> /Alimentación/5Vin
- J901 pad 2: 5V -> /Alimentación/5Vin
- U101 pad 119: /Sensores/GNSS_Tx -> /Conexiones_extra/UARTA_TX
- U101 pad 122: /Sensores/GNSS_Rx -> /Conexiones_extra/UARTA_RX
- U101 pad 124: /Conexiones_extra/UARTA_RX -> /Conexiones_extra/UARTB_RX
- U101 pad 129: /Conexiones_extra/UARTA_TX -> /Conexiones_extra/UARTB_TX
- U101 pad 141: /Conexiones_extra/UARTD_RX -> /Conexiones_extra/UARTC_RX
- U101 pad 142: /Conexiones_extra/UARTD_TX -> /Conexiones_extra/UARTC_TX
- U101 pad 2: /MCU/PE_3(EXTI3) -> unconnected-(U101-Pad2)
- U101 pad 28: /Alimentación/I_MEAS -> unconnected-(U101-Pad28)
- U101 pad 29: /Alimentación/V_MEAS -> unconnected-(U101-Pad29)
- U101 pad 40: unconnected-(U101-Pad40) -> /Alimentación/I_MEAS
- U101 pad 41: unconnected-(U101-Pad41) -> /Alimentación/V_MEAS
- U101 pad 56: /Sensores/MAG_INT_DATA_RDY -> unconnected-(U101-Pad56)
- U101 pad 68: /MCU/PE_15(EXTI15) -> /Sensores/MAG_INT_DATA_RDY
- U101 pad 77: /MCU/USART3_TX -> /Sensores/GNSS_Tx
- U101 pad 78: /MCU/USART3_RX -> /Sensores/GNSS_Rx
- U101 pad 87: unconnected-(U101-Pad87) -> /MCU/PG_2(EXTI2)
- U201 pad 4: /MCU/PE_3(EXTI3) -> /MCU/PG_2(EXTI2)
- U901 pad 3: /Alimentación/5Vin -> 5V
Routing:
- net /Conexiones_extra/UARTC_TX: track 0.00 -> 93.3 mm, vias 0 -> 1
- net /Conexiones_extra/UARTC_RX: track 0.00 -> 90.5 mm, vias 0 -> 1
- net /MCU/PD_10(EXTI10): track 0.00 -> 81.9 mm, vias 0 -> 3
- net /MCU/UART7_RX: track 0.00 -> 77.2 mm, vias 0 -> 4
- net Net-(C906-Pad1): track 0.00 -> 76.3 mm, vias 0 -> 2
- net Net-(C907-Pad1): track 0.00 -> 76.0 mm, vias 0 -> 2
- net /Conexiones_extra/UARTA_TX: track 0.00 -> 69.0 mm, vias 0 -> 1
- net /Conexiones_extra/UARTB_TX: track 0.00 -> 68.6 mm, vias 0 -> 1
- net /Conexiones_extra/UARTA_RX: track 0.00 -> 67.4 mm, vias 0 -> 1
- net /Conexiones_extra/UARTB_RX: track 0.00 -> 63.0 mm, vias 0 -> 1
- net /MCU/USART3_RX: track 33.3 -> 0.00 mm, vias 2 -> 0
- net 3V3: track 82.7 -> 52.2 mm, vias 0 -> 3
- net /Sensores/GNSS_SDA: track 83.9 -> 111.5 mm, vias 3 -> 4
- net /MCU/TIM2_CH2: track 20.4 -> 47.2 mm
- net /MCU/TIM2_CH3: track 20.8 -> 47.4 mm
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
Commit message: positioning of componentes 80x80 pcb
Parts:
- removed C1101, C1102: 100nF, Capacitor_SMD:C_0402_1005Metric_Pad0.74x0.62mm_HandSolder
- removed C116: 4.7uF, Capacitor_SMD:C_0603_1608Metric_Pad1.08x0.95mm_HandSolder
- removed C119: 100nF, Capacitor_SMD:C_0603_1608Metric_Pad1.08x0.95mm_HandSolder
- removed C901: 1.6u, Capacitor_SMD:C_0603_1608Metric_Pad1.08x0.95mm_HandSolder
- removed C902: 0.1u, Capacitor_SMD:C_0603_1608Metric_Pad1.08x0.95mm_HandSolder
- removed D1101, D1102: LED_RED, LED_SMD:LED_0805_2012Metric_Pad1.15x1.40mm_HandSolder
- removed D1103, D1104: LED_GREEN, LED_SMD:LED_0805_2012Metric_Pad1.15x1.40mm_HandSolder
- removed D1105, D1106: LED_YELLOW, LED_SMD:LED_0805_2012Metric_Pad1.15x1.40mm_HandSolder
- removed D1107, D1108: LED_BLUE, LED_SMD:LED_0805_2012Metric_Pad1.15x1.40mm_HandSolder
- removed D901: PMEG60T30ELRX, PMEG60T30ELRX:SODFL3517X110N
- removed J601: SWD Debug Connector, Connector_PinHeader_2.54mm:PinHeader_2x03_P2.54mm_Vertical
- removed J802: CAN 1 Connector 2, DF13A-3P-1.25H(21):HRS_DF13A-3P-1.25H(21)
- removed J804: CAN 2 Connector 2, DF13A-3P-1.25H(21):HRS_DF13A-3P-1.25H(21)
- removed Q1101, Q1102, Q1103, Q1104, Q1105, Q1106, Q1107, Q1108: 2N7002, Package_TO_SOT_SMD:SOT-23
- removed Q901: Q_PMOS_GSD, Package_TO_SOT_SMD:SOT-23
- removed R1101, R1102, R1104, R1105, R1107, R1108, R1110, R1111, R1113, R1114, R1116, R1117, R1119, R1120, R1122, R1123, R1125, R1126: R, Resistor_SMD:R_0402_1005Metric_Pad0.72x0.64mm_HandSolder
- removed R1103, R1106, R1109, R1112, R1115, R1118, R1121, R1124: R, Resistor_SMD:R_0805_2012Metric_Pad1.20x1.40mm_HandSolder
- removed R901: 10, Resistor_SMD:R_0603_1608Metric_Pad0.98x0.95mm_HandSolder
- removed R902: 6.8k, Resistor_SMD:R_0603_1608Metric_Pad0.98x0.95mm_HandSolder
- removed R903: 33, Resistor_SMD:R_0603_1608Metric_Pad0.98x0.95mm_HandSolder
- removed SW101: SW RESET, Button_Switch_SMD:SW_SPST_TL3305A
- removed SW1101, SW1102: SW Propósito General, Button_Switch_SMD:SW_SPST_TL3305A
- C701: footprint Capacitor_SMD:C_0603_1608Metric_Pad1.08x0.95mm_HandSolder -> Capacitor_SMD:C_0402_1005Metric_Pad0.74x0.62mm_HandSolder; moved to B.Cu
- C702, C801, C802, C804, C805, C906, C907, D801, D802, J701, J801, J803, R103, R104, R107, R108, R701, R705, R706, R904, R905, R906, R907, U801, U802: moved to B.Cu
- moved R904 158.1 mm to (124.7, 114.0), turned to 90 degrees
- moved R905 153.2 mm to (120.7, 114.0), turned to 90 degrees
- moved C906 151.3 mm to (125.8, 114.1), turned to 90 degrees
- moved C907 148.9 mm to (119.5, 114.0), turned to 90 degrees
- moved C109 59.9 mm to (142.3, 89.0), turned to -90 degrees
- moved C108 59.0 mm to (142.1, 101.9), turned to -90 degrees
- moved R701 51.6 mm to (129.7, 102.5), turned to -90 degrees
- moved C111 46.5 mm to (140.3, 76.0), turned to 0 degrees
- moved C114 41.2 mm to (140.6, 110.7), turned to 0 degrees
- moved R108 40.2 mm to (123.2, 102.2), turned to 0 degrees
- moved R806 39.8 mm to (158.6, 78.4), turned to 0 degrees
- moved R107 39.2 mm to (123.3, 101.1), turned to 180 degrees
- moved C112 35.8 mm to (118.5, 85.4)
- moved R807 33.2 mm to (157.7, 95.2)
- moved J801 31.3 mm to (130.8, 73.1), turned to 180 degrees
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Routing:
- net 5V: track 128.3 -> 0.00 mm
- net /Sensores/GNSS_SDA: track 111.5 -> 0.00 mm, vias 4 -> 0
- net /Sensores/GNSS_SCL: track 108.2 -> 0.00 mm, vias 4 -> 0
- net /Conexiones_extra/SPI_MISO: track 103.2 -> 0.00 mm, vias 1 -> 0
- net /Conexiones_extra/SPI_EOC: track 102.3 -> 0.00 mm, vias 1 -> 0
- net /Conexiones_extra/SPI_MOSI: track 100.8 -> 0.00 mm, vias 1 -> 0
- net /Conexiones_extra/SPI_CS: track 100.7 -> 0.00 mm, vias 1 -> 0
- net /Conexiones_extra/SPI_SCK: track 99.8 -> 0.00 mm, vias 1 -> 0
- net /Sensores/GNSS_Rx: track 95.2 -> 0.00 mm, vias 4 -> 0
- net /Conexiones_extra/UARTC_TX: track 93.3 -> 0.00 mm, vias 1 -> 0
- net /Sensores/GNSS_Tx: track 91.6 -> 0.00 mm, vias 4 -> 0
- net /Conexiones_extra/UARTC_RX: track 90.5 -> 0.00 mm, vias 1 -> 0
- net /Sensores/MAG_INT_DATA_RDY: track 88.8 -> 0.00 mm, vias 3 -> 0
- net /Conexiones_extra/I2CA_SCL: track 87.2 -> 0.00 mm, vias 1 -> 0
- net /Conexiones_extra/I2CA_SDA: track 82.0 -> 0.00 mm, vias 1 -> 0
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Other:
- board size 100 x 80 mm -> 80 x 80 mm
