File: hardware/Drone FCC/Drone FCC.kicad_pcb (KiCad board)
At the start: 4 copper layers, 80 x 80 mm, 110 parts, among them J1 Conn_02x06_Odd_Even, J1001 SPI externo, J1003 I2C externo x2, J1005 5V y 3V3 x 2, J201 Mag Dupont, J202 Mag DF13, J203 GPS Dupont, J204 GPS M8N - DF13, J301 ESC 1, J302 ESC 2, J303 ESC 3, J304 ESC 4, J305 ESC 5, J306 ESC 6, J307 ESC 7, J308 ESC 8, J309 SERVO 1, J310 SERVO 2, J311 SERVO 3, J312 SERVO 4, J313 Power Servo, J401 DSM Spektrum JST, J402 PPM Dupont, J501 Micro USB - B, J701 DM3AT-SF-PEJM5, J801 CAN 1 Connector 1, J803 CAN 2 Connector 1, J901 PM02 PixHawk, U101 STM32F746ZGTx, U201 ICM-42688-V, U202 ILPS22QSTR, U501 USBLC6-2SC6, U801 SN65HVD230, U802 SN65HVD230, U901 ZLDO1117QG33TA, Y101 12MHz, Y102 32.768kHz

Commit message: positioned components in 100x60 board with incomplete routing
Parts:
- added C1101: 100nF, Capacitor_SMD:C_0402_1005Metric_Pad0.74x0.62mm_HandSolder, F.Cu at (-19.8, 18.0)
- added C1102: 100nF, Capacitor_SMD:C_0402_1005Metric_Pad0.74x0.62mm_HandSolder, F.Cu at (-23.0, 21.3)
- added C116: 4.7uF, Capacitor_SMD:C_0603_1608Metric_Pad1.08x0.95mm_HandSolder, F.Cu at (31.2, 24.6)
- added C119: 100nF, Capacitor_SMD:C_0603_1608Metric_Pad1.08x0.95mm_HandSolder, F.Cu at (-136.1, 50.2)
- added C901: 1.6u, Capacitor_SMD:C_0603_1608Metric_Pad1.08x0.95mm_HandSolder, F.Cu at (-35.4, 43.4)
- added C902: 0.1u, Capacitor_SMD:C_0603_1608Metric_Pad1.08x0.95mm_HandSolder, F.Cu at (-25.5, 36.4)
- added D1101: LED_RED, LED_SMD:LED_0805_2012Metric_Pad1.15x1.40mm_HandSolder, F.Cu at (-33.4, 18.1)
- added D1102: LED_RED, LED_SMD:LED_0805_2012Metric_Pad1.15x1.40mm_HandSolder, F.Cu at (-18.2, 1.57)
- added D1103: LED_GREEN, LED_SMD:LED_0805_2012Metric_Pad1.15x1.40mm_HandSolder, F.Cu at (-33.3, 14.9)
- added D1104: LED_GREEN, LED_SMD:LED_0805_2012Metric_Pad1.15x1.40mm_HandSolder, F.Cu at (-38.2, 21.2)
- added D1105: LED_YELLOW, LED_SMD:LED_0805_2012Metric_Pad1.15x1.40mm_HandSolder, F.Cu at (-38.2, 18.1)
- added D1106: LED_YELLOW, LED_SMD:LED_0805_2012Metric_Pad1.15x1.40mm_HandSolder, F.Cu at (-23.0, 1.57)
- added D1107: LED_BLUE, LED_SMD:LED_0805_2012Metric_Pad1.15x1.40mm_HandSolder, F.Cu at (-23.0, 4.61)
- added D1108: LED_BLUE, LED_SMD:LED_0805_2012Metric_Pad1.15x1.40mm_HandSolder, F.Cu at (-27.9, 10.5)
- added D901: PMEG60T30ELRX, PMEG60T30ELRX:SODFL3517X110N, F.Cu at (-40.3, 43.8)
- added J601: SWD Debug Connector, Connector_PinHeader_2.54mm:PinHeader_2x03_P2.54mm_Vertical, F.Cu at (-6.04, 2.37)
- added Q1101: 2N7002, Package_TO_SOT_SMD:SOT-23, F.Cu at (-43.1, 18.8)
- added Q1102: 2N7002, Package_TO_SOT_SMD:SOT-23, F.Cu at (-27.9, 6.72)
- added Q1103: 2N7002, Package_TO_SOT_SMD:SOT-23, F.Cu at (-32.7, 2.27)
- added Q1104: 2N7002, Package_TO_SOT_SMD:SOT-23, F.Cu at (-27.9, 2.27)
- added Q1105: 2N7002, Package_TO_SOT_SMD:SOT-23, F.Cu at (-32.7, 11.2)
- added Q1106: 2N7002, Package_TO_SOT_SMD:SOT-23, F.Cu at (-43.1, 14.4)
- added Q1107: 2N7002, Package_TO_SOT_SMD:SOT-23, F.Cu at (-32.7, 6.72)
- added Q1108: 2N7002, Package_TO_SOT_SMD:SOT-23, F.Cu at (-38.2, 14.4)
- added Q901: Q_PMOS_GSD, Package_TO_SOT_SMD:SOT-23, F.Cu at (-21.0, 28.6)
- added R1101: R, Resistor_SMD:R_0402_1005Metric_Pad0.72x0.64mm_HandSolder, F.Cu at (-13.3, 12.0)
- added R1102: R, Resistor_SMD:R_0402_1005Metric_Pad0.72x0.64mm_HandSolder, F.Cu at (-14.2, 1.04)
- added R1103: R, Resistor_SMD:R_0805_2012Metric_Pad1.20x1.40mm_HandSolder, F.Cu at (-23.1, 10.6)
- added R1104: R, Resistor_SMD:R_0402_1005Metric_Pad0.72x0.64mm_HandSolder, F.Cu at (-16.6, 12.0)
- added R1105: R, Resistor_SMD:R_0402_1005Metric_Pad0.72x0.64mm_HandSolder, F.Cu at (-43.9, 22.0)
- added R1106: R, Resistor_SMD:R_0805_2012Metric_Pad1.20x1.40mm_HandSolder, F.Cu at (-28.7, 17.9)
- added R1107: R, Resistor_SMD:R_0402_1005Metric_Pad0.72x0.64mm_HandSolder, F.Cu at (-15.8, 9.98)
- added R1108: R, Resistor_SMD:R_0402_1005Metric_Pad0.72x0.64mm_HandSolder, F.Cu at (-18.2, 16.0)
- added R1109: R, Resistor_SMD:R_0805_2012Metric_Pad1.20x1.40mm_HandSolder, F.Cu at (-18.2, 4.56)
- added R1110: R, Resistor_SMD:R_0402_1005Metric_Pad0.72x0.64mm_HandSolder, F.Cu at (-26.2, 22.4)
- added R1111: R, Resistor_SMD:R_0402_1005Metric_Pad0.72x0.64mm_HandSolder, F.Cu at (-29.5, 20.6)
- added R1112: R, Resistor_SMD:R_0805_2012Metric_Pad1.20x1.40mm_HandSolder, F.Cu at (-23.8, 13.5)
- added R1113: R, Resistor_SMD:R_0402_1005Metric_Pad0.72x0.64mm_HandSolder, F.Cu at (-14.2, 5.02)
- added R1114: R, Resistor_SMD:R_0402_1005Metric_Pad0.72x0.64mm_HandSolder, F.Cu at (-19.8, 13.0)
- added R1115: R, Resistor_SMD:R_0805_2012Metric_Pad1.20x1.40mm_HandSolder, F.Cu at (-18.2, 7.51)
- added R1116: R, Resistor_SMD:R_0402_1005Metric_Pad0.72x0.64mm_HandSolder, F.Cu at (-14.2, 3.03)
- added R1117: R, Resistor_SMD:R_0402_1005Metric_Pad0.72x0.64mm_HandSolder, F.Cu at (-14.2, 7.01)
- added R1118: R, Resistor_SMD:R_0805_2012Metric_Pad1.20x1.40mm_HandSolder, F.Cu at (-33.5, 21.1)
- added R1119: R, Resistor_SMD:R_0402_1005Metric_Pad0.72x0.64mm_HandSolder, F.Cu at (-19.0, 9.98)
- added R1120: R, Resistor_SMD:R_0402_1005Metric_Pad0.72x0.64mm_HandSolder, F.Cu at (-26.2, 20.4)
- added R1121: R, Resistor_SMD:R_0805_2012Metric_Pad1.20x1.40mm_HandSolder, F.Cu at (-23.0, 7.60)
- added R1122: R, Resistor_SMD:R_0402_1005Metric_Pad0.72x0.64mm_HandSolder, F.Cu at (-16.6, 14.0)
- added R1123: R, Resistor_SMD:R_0402_1005Metric_Pad0.72x0.64mm_HandSolder, F.Cu at (-23.0, 19.3)
- added R1124: R, Resistor_SMD:R_0805_2012Metric_Pad1.20x1.40mm_HandSolder, F.Cu at (-28.6, 14.9)
- added R1125: R, Resistor_SMD:R_0402_1005Metric_Pad0.72x0.64mm_HandSolder, F.Cu at (-21.4, 16.0)
- added R1126: R, Resistor_SMD:R_0402_1005Metric_Pad0.72x0.64mm_HandSolder, F.Cu at (-24.7, 17.3)
- added R901: 10, Resistor_SMD:R_0603_1608Metric_Pad0.98x0.95mm_HandSolder, F.Cu at (-31.0, 38.4)
- added R902: 6.8k, Resistor_SMD:R_0603_1608Metric_Pad0.98x0.95mm_HandSolder, F.Cu at (-35.4, 45.9)
- added R903: 33, Resistor_SMD:R_0603_1608Metric_Pad0.98x0.95mm_HandSolder, F.Cu at (-25.5, 33.9)
- added SW101: SW RESET, Button_Switch_SMD:SW_SPST_TL3305A, F.Cu at (-133.1, 41.5)
- added SW1101: SW Propósito General, Button_Switch_SMD:SW_SPST_TL3305A, F.Cu at (-40.4, 9.12)
- added SW1102: SW Propósito General, Button_Switch_SMD:SW_SPST_TL3305A, F.Cu at (-40.4, 3.07)
- C701, C702, C801, C802, C804, C805, C906, C907, D801, D802, J701, J801, J803, R103, R104, R107, R108, R701, R702, R703, R704, R705, R706, R904, R905, R906, R907, U801, U802: moved to F.Cu
- J1: value Conn_02x06_Odd_Even -> UARTs externo x 3
- moved C204 310.7 mm to (-157.8, 89.9), turned to 0 degrees
- moved C205 305.2 mm to (-154.6, 89.9), turned to 0 degrees
- moved U202 297.8 mm to (-144.8, 89.4), turned to 0 degrees
- moved C206 293.7 mm to (-144.2, 85.8), turned to 0 degrees
- moved R106 287.5 mm to (-131.0, 48.0), turned to 0 degrees
- moved C203 283.0 mm to (-132.6, 78.2)
- moved R105 281.3 mm to (-126.6, 45.5), turned to 0 degrees
- moved C201 279.7 mm to (-126.0, 70.5), turned to 0 degrees
- moved R103 274.9 mm to (-143.7, 63.8), turned to 0 degrees
- moved R104 261.5 mm to (-121.5, 39.5)
- moved C702 248.4 mm to (-108.2, 64.1), turned to 0 degrees
- moved R704 235.4 mm to (-92.3, 39.5), turned to 0 degrees
- moved R705 232.9 mm to (-89.1, 39.5), turned to 0 degrees
- moved R706 232.7 mm to (-89.1, 41.5), turned to 0 degrees
- moved R702 231.5 mm to (-92.3, 41.5), turned to 0 degrees
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Connections:
- net Net-(D801-Pad1) renamed /Interfaz_CAN/CAN-
- net Net-(D801-Pad2) renamed /Interfaz_CAN/CAN+
- J1 pad 1: /Conexiones_extra/UARTB_RX -> /Conexiones_extra/UARTC_RX
- J1 pad 10: 3V3 -> /Conexiones_extra/UARTA_TX
- J1 pad 11: /Conexiones_extra/UARTC_TX -> 3V3
- J1 pad 2: 3V3 -> /Conexiones_extra/UARTC_TX
- J1 pad 3: /Conexiones_extra/UARTB_TX -> 3V3
- J1 pad 5: /Conexiones_extra/UARTA_RX -> /Conexiones_extra/UARTB_RX
- J1 pad 6: 3V3 -> /Conexiones_extra/UARTB_TX
- J1 pad 7: /Conexiones_extra/UARTA_TX -> 3V3
- J1 pad 9: /Conexiones_extra/UARTC_RX -> /Conexiones_extra/UARTA_RX
- J1001 pad 2: /Conexiones_extra/SPI_EOC -> 3V3
- J1001 pad 3: /Conexiones_extra/SPI_SCK -> /Conexiones_extra/SPI_EOC
- J1001 pad 4: /Conexiones_extra/SPI_CS -> GND
- J1001 pad 5: /Conexiones_extra/SPI_MOSI -> /Conexiones_extra/SPI_CS
- J1001 pad 6: /Conexiones_extra/SPI_MISO -> /Conexiones_extra/SPI_SCK
- J1001 pad 7: 3V3 -> /Conexiones_extra/SPI_MISO
- J1001 pad 8: GND -> /Conexiones_extra/SPI_MOSI
- J1003 pad 1: /Conexiones_extra/I2CA_SCL -> 5V
- J1003 pad 10: /Conexiones_extra/I2CA_SDA -> /Conexiones_extra/I2CA_SCL
- J1003 pad 2: /Conexiones_extra/I2CA_SCL -> 3V3
- J1003 pad 7: 5V -> /Conexiones_extra/I2CA_SDA
- J1003 pad 8: 3V3 -> /Conexiones_extra/I2CA_SDA
- J1003 pad 9: /Conexiones_extra/I2CA_SDA -> /Conexiones_extra/I2CA_SCL
- J201 pad 3: unconnected-(J201-Pad3) -> /Sensores/GNSS_SDA
- J201 pad 6: /Sensores/GNSS_SDA -> unconnected-(J201-Pad6)
- J203 pad 1: /Sensores/GNSS_Tx -> /Sensores/GNSS_Rx
- J203 pad 2: /Sensores/GNSS_Rx -> /Sensores/GNSS_PPS
- J203 pad 3: GND -> /Sensores/GNSS_Tx
- J203 pad 6: /MCU/PD_10(EXTI10) -> GND
- J204 pad 4: /Sensores/GNSS_SCL -> /Sensores/GNSS_PPS
- J204 pad 5: /Sensores/GNSS_SDA -> unconnected-(J204-Pad5)
- J309 pad 1: /MCU/TIM2_CH1 -> /MCU/TIM4_CH1
- J310 pad 1: /MCU/TIM2_CH2 -> /MCU/TIM4_CH2
- J311 pad 1: /MCU/TIM2_CH3 -> /MCU/TIM4_CH3
- J312 pad 1: /MCU/TIM2_CH4 -> /MCU/TIM4_CH4
- J401 pad 3: /MCU/UART7_RX -> /RC control/DSM_DATA
- J402 pad 3: /MCU/TIM4_CH1 -> /MCU/TIM8_CH2
- U101 pad 119: /Conexiones_extra/UARTA_TX -> /Conexiones_extra/UARTC_TX
- U101 pad 122: /Conexiones_extra/UARTA_RX -> /Conexiones_extra/UARTC_RX
- U101 pad 141: /Conexiones_extra/UARTC_RX -> /MCU/UART8_RX
- U101 pad 142: /Conexiones_extra/UARTC_TX -> /MCU/UART8_TX
- U101 pad 34: /MCU/TIM2_CH1 -> unconnected-(U101-Pad34)
- U101 pad 35: /MCU/TIM2_CH2 -> /Alimentación/I_MEAS
- U101 pad 36: /MCU/TIM2_CH3 -> /Alimentación/V_MEAS
- U101 pad 4: unconnected-(U101-Pad4) -> /MCU/TIM9_CH1
- U101 pad 40: /Alimentación/I_MEAS -> unconnected-(U101-Pad40)
- U101 pad 41: /Alimentación/V_MEAS -> /Sensores/GNSS_PPS
- U101 pad 57: unconnected-(U101-Pad57) -> /Sensores/MAG_INT_DATA_RDY
- U101 pad 58: /MCU/UART7_RX -> /Sensores/GNSS_Rx
- U101 pad 59: unconnected-(U101-Pad59) -> /Sensores/GNSS_Tx
- U101 pad 68: /Sensores/MAG_INT_DATA_RDY -> /MCU/PE_15(EXTI15)
- U101 pad 77: /Sensores/GNSS_Tx -> /Conexiones_extra/UARTA_TX
- U101 pad 78: /Sensores/GNSS_Rx -> /Conexiones_extra/UARTA_RX
- U101 pad 97: unconnected-(U101-Pad97) -> /MCU/TIM8_CH2
Routing:
- net 5V: track 0.00 -> 151.9 mm
- net /Sensores/GNSS_PPS: track 0.00 -> 45.6 mm, vias 0 -> 2
- net /MCU/TIM1_CH4: track 0.00 -> 44.6 mm, vias 0 -> 1
- net /MCU/TIM1_CH3: track 0.00 -> 43.8 mm, vias 0 -> 1
- net /MCU/TIM1_CH2: track 0.00 -> 43.2 mm, vias 0 -> 1
- net Net-(C906-Pad1): track 0.00 -> 43.1 mm, vias 0 -> 2
- net Net-(C907-Pad1): track 0.00 -> 42.2 mm, vias 0 -> 2
- net /MCU/TIM3_CH1: track 0.00 -> 42.2 mm, vias 0 -> 1
- net /MCU/TIM3_CH2: track 0.00 -> 41.4 mm, vias 0 -> 1
- net /MCU/TIM1_CH1: track 0.00 -> 41.0 mm, vias 0 -> 1
- net /MCU/TIM3_CH3: track 0.00 -> 40.6 mm, vias 0 -> 1
- net /MCU/TIM3_CH4: track 0.00 -> 39.9 mm, vias 0 -> 1
- net /Conexiones_extra/I2CA_SDA: track 0.00 -> 34.4 mm, vias 0 -> 1
- net /Conexiones_extra/I2CA_SCL: track 0.00 -> 32.4 mm, vias 0 -> 1
- net /MCU/SDMMC1_D0: track 0.00 -> 26.1 mm, vias 0 -> 2
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- removed copper zone on In2.Cu, net 3V3
- removed copper zone on In1.Cu, net GND
Other:
- board size 80 x 80 mm -> 60 x 100 mm
