File: hardware/Drone FCC/conexiones_extra.kicad_sch (KiCad schematic)
At the start: 5 parts

Commit message: re enumeration of components
Parts:
- J1001, J1002, J1004, J1005: renamed from J?; footprint (none) -> Connector_PinHeader_2.54mm:PinHeader_2x04_P2.54mm_Horizontal
- J1003: renamed from J?; footprint (none) -> Connector_PinHeader_2.54mm:PinHeader_2x05_P2.54mm_Horizontal
Changed lines of the file:
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@@
   (symbol (lib_id "Connector_Generic:Conn_02x05_Odd_Even") (at 62.23 70.485 0) (unit 1)
     (in_bom yes) (on_board yes)
-    (property "Reference" "J?" (id 0) (at 63.5 58.42 0))
+    (property "Reference" "J1003" (id 0) (at 63.5 58.42 0))
     (property "Value" "I2C externo x2" (id 1) (at 63.5 60.96 0))
-    (property "Footprint" "" (id 2) (at 62.23 70.485 0)
+    (property "Footprint" "Connector_PinHeader_2.54mm:PinHeader_2x05_P2.54mm_Horizontal" (id 2) (at 62.23 70.485 0)
       (effects (font (size 1.27 1.27)) hide)
     )
@@
   (symbol (lib_id "power:GND") (at 153.035 102.87 0) (unit 1)
     (in_bom yes) (on_board yes) (fields_autoplaced)
-    (property "Reference" "#PWR?" (id 0) (at 153.035 109.22 0)
+    (property "Reference" "#PWR0174" (id 0) (at 153.035 109.22 0)
       (effects (font (size 1.27 1.27)) hide)
     )
@@
   (symbol (lib_id "power:GND") (at 153.035 40.64 0) (unit 1)
     (in_bom yes) (on_board yes) (fields_autoplaced)
-    (property "Reference" "#PWR?" (id 0) (at 153.035 46.99 0)
+    (property "Reference" "#PWR0166" (id 0) (at 153.035 46.99 0)
       (effects (font (size 1.27 1.27)) hide)
     )
@@
   (symbol (lib_id "Connector_Generic:Conn_02x04_Odd_Even") (at 62.23 33.02 0) (unit 1)
     (in_bom yes) (on_board yes) (fields_autoplaced)
-    (property "Reference" "J?" (id 0) (at 63.5 23.495 0))
+    (property "Reference" "J1001" (id 0) (at 63.5 23.495 0))
     (property "Value" "SPI externo" (id 1) (at 63.5 26.035 0))
-    (property "Footprint" "" (id 2) (at 62.23 33.02 0)
+    (property "Footprint" "Connector_PinHeader_2.54mm:PinHeader_2x04_P2.54mm_Horizontal" (id 2) (at 62.23 33.02 0)
       (effects (font (size 1.27 1.27)) hide)
     )
@@
   (symbol (lib_id "power:GND") (at 83.82 40.64 0) (unit 1)
     (in_bom yes) (on_board yes) (fields_autoplaced)
-    (property "Reference" "#PWR?" (id 0) (at 83.82 46.99 0)
+    (property "Reference" "#PWR0172" (id 0) (at 83.82 46.99 0)
       (effects (font (size 1.27 1.27)) hide)
     )
@@
   (symbol (lib_id "power:GND") (at 43.18 75.565 0) (mirror y) (unit 1)
     (in_bom yes) (on_board yes) (fields_autoplaced)
-    (property "Reference" "#PWR?" (id 0) (at 43.18 81.915 0)
+    (property "Reference" "#PWR0171" (id 0) (at 43.18 81.915 0)
       (effects (font (size 1.27 1.27)) hide)
     )
@@
   (symbol (lib_id "power:GND") (at 112.395 69.215 0) (mirror y) (unit 1)
     (in_bom yes) (on_board yes) (fields_autoplaced)
-    (property "Reference" "#PWR?" (id 0) (at 112.395 75.565 0)
+    (property "Reference" "#PWR0167" (id 0) (at 112.395 75.565 0)
       (effects (font (size 1.27 1.27)) hide)
     )
@@
   (symbol (lib_id "Connector_Generic:Conn_02x04_Odd_Even") (at 131.445 61.595 0) (unit 1)
     (in_bom yes) (on_board yes) (fields_autoplaced)
-    (property "Reference" "J?" (id 0) (at 132.715 52.705 0))
+    (property "Reference" "J1004" (id 0) (at 132.715 52.705 0))
     (property "Value" "UART externa x2" (id 1) (at 132.715 55.245 0))
-    (property "Footprint" "" (id 2) (at 131.445 61.595 0)
+    (property "Footprint" "Connector_PinHeader_2.54mm:PinHeader_2x04_P2.54mm_Horizontal" (id 2) (at 131.445 61.595 0)
       (effects (font (size 1.27 1.27)) hide)
     )
@@
   (symbol (lib_id "Connector_Generic:Conn_02x04_Odd_Even") (at 131.445 33.02 0) (unit 1)
     (in_bom yes) (on_board yes) (fields_autoplaced)
-    (property "Reference" "J?" (id 0) (at 132.715 24.13 0))
+    (property "Reference" "J1002" (id 0) (at 132.715 24.13 0))
     (property "Value" "UART externa x2" (id 1) (at 132.715 26.67 0))
-    (property "Footprint" "" (id 2) (at 131.445 33.02 0)
+    (property "Footprint" "Connector_PinHeader_2.54mm:PinHeader_2x04_P2.54mm_Horizontal" (id 2) (at 131.445 33.02 0)
       (effects (font (size 1.27 1.27)) hide)
     )
@@
   (symbol (lib_id "Connector_Generic:Conn_02x04_Odd_Even") (at 131.445 97.79 0) (unit 1)
     (in_bom yes) (on_board yes) (fields_autoplaced)
-    (property "Reference" "J?" (id 0) (at 132.715 88.9 0))
+    (property "Reference" "J1005" (id 0) (at 132.715 88.9 0))
     (property "Value" "5V y 3V3 x 2" (id 1) (at 132.715 91.44 0))
-    (property "Footprint" "" (id 2) (at 131.445 97.79 0)
+    (property "Footprint" "Connector_PinHeader_2.54mm:PinHeader_2x04_P2.54mm_Horizontal" (id 2) (at 131.445 97.79 0)
       (effects (font (size 1.27 1.27)) hide)
     )
@@
   (symbol (lib_id "power:GND") (at 153.035 69.215 0) (unit 1)
     (in_bom yes) (on_board yes) (fields_autoplaced)
-    (property "Reference" "#PWR?" (id 0) (at 153.035 75.565 0)
+    (property "Reference" "#PWR0168" (id 0) (at 153.035 75.565 0)
       (effects (font (size 1.27 1.27)) hide)
     )
@@
   (symbol (lib_id "power:GND") (at 83.82 75.565 0) (unit 1)
     (in_bom yes) (on_board yes) (fields_autoplaced)
-    (property "Reference" "#PWR?" (id 0) (at 83.82 81.915 0)
+    (property "Reference" "#PWR0170" (id 0) (at 83.82 81.915 0)
       (effects (font (size 1.27 1.27)) hide)
     )
@@
   (symbol (lib_id "power:GND") (at 112.395 102.87 0) (mirror y) (unit 1)
     (in_bom yes) (on_board yes) (fields_autoplaced)
-    (property "Reference" "#PWR?" (id 0) (at 112.395 109.22 0)
+    (property "Reference" "#PWR0173" (id 0) (at 112.395 109.22 0)
       (effects (font (size 1.27 1.27)) hide)
     )
@@
   (symbol (lib_id "power:GND") (at 112.395 40.64 0) (mirror y) (unit 1)
     (in_bom yes) (on_board yes) (fields_autoplaced)
-    (property "Reference" "#PWR?" (id 0) (at 112.395 46.99 0)
-      (effects (font (size 1.27 1.27)) hide)
-    )
+    (property "Reference" "#PWR0169" (id 0) (at 112.395 46.99 0)
+      (effects (font (size 1.27 1.27)) hide)
+    )

Commit message: continued preliminar routing
Connections:
- net 3V3: now also J1003.9 (Pin_9); no longer J1003.8 (Pin_8)
- net 5V: now also J1001.1 (Pin_1), J1003.1 (Pin_1), J1003.3 (Pin_3); no longer J1001.8 (Pin_8), J1003.10 (Pin_10), J1003.9 (Pin_9)
- net GND: now also J1001.8 (Pin_8); no longer J1001.6 (Pin_6)
- net I2CA_SCL: now also J1003.8 (Pin_8); no longer J1003.1 (Pin_1)
- net I2CA_SDA: now also J1003.10 (Pin_10); no longer J1003.3 (Pin_3)
- net SPI_SCK: now also J1001.6 (Pin_6); no longer J1001.1 (Pin_1)
Changed lines of the file:
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@@
   (junction (at 112.395 100.33) (diameter 0) (color 0 0 0 0)
   )
-  (wire (pts (xy 83.82 70.485) (xy 83.82 75.565))
+  (wire (pts (xy 86.995 70.485) (xy 86.995 75.565))
     (stroke (width 0) (type default) (color 0 0 0 0))
   )
@@
     (stroke (width 0) (type default) (color 0 0 0 0))
   )
-  (wire (pts (xy 83.82 35.56) (xy 83.82 40.64))
-    (stroke (width 0) (type default) (color 0 0 0 0))
-  )
   (wire (pts (xy 126.365 97.79) (xy 112.395 97.79))
     (stroke (width 0) (type default) (color 0 0 0 0))
@@
     (stroke (width 0) (type default) (color 0 0 0 0))
   )
+  (wire (pts (xy 74.93 75.565) (xy 69.85 75.565))
+    (stroke (width 0) (type default) (color 0 0 0 0))
+  )
   (wire (pts (xy 52.07 67.945) (xy 57.15 67.945))
     (stroke (width 0) (type default) (color 0 0 0 0))
@@
     (stroke (width 0) (type default) (color 0 0 0 0))
   )
-  (wire (pts (xy 69.85 38.1) (xy 74.93 38.1))
+  (wire (pts (xy 69.85 38.1) (xy 83.82 38.1))
     (stroke (width 0) (type default) (color 0 0 0 0))
   )
@@
     (stroke (width 0) (type default) (color 0 0 0 0))
   )
-  (wire (pts (xy 54.61 75.565) (xy 57.15 75.565))
+  (wire (pts (xy 52.07 75.565) (xy 57.15 75.565))
     (stroke (width 0) (type default) (color 0 0 0 0))
   )
@@
     (stroke (width 0) (type default) (color 0 0 0 0))
   )
-  (wire (pts (xy 76.835 73.025) (xy 69.85 73.025))
-    (stroke (width 0) (type default) (color 0 0 0 0))
-  )
   (wire (pts (xy 43.18 70.485) (xy 43.18 75.565))
     (stroke (width 0) (type default) (color 0 0 0 0))
   )
-  (wire (pts (xy 69.85 70.485) (xy 83.82 70.485))
+  (wire (pts (xy 83.82 38.1) (xy 83.82 40.64))
+    (stroke (width 0) (type default) (color 0 0 0 0))
+  )
+  (wire (pts (xy 69.85 70.485) (xy 86.995 70.485))
     (stroke (width 0) (type default) (color 0 0 0 0))
   )
@@
     (stroke (width 0) (type default) (color 0 0 0 0))
   )
+  (wire (pts (xy 69.85 35.56) (xy 74.93 35.56))
+    (stroke (width 0) (type default) (color 0 0 0 0))
+  )
   (wire (pts (xy 139.065 97.79) (xy 153.035 97.79))
     (stroke (width 0) (type default) (color 0 0 0 0))
@@
     (stroke (width 0) (type default) (color 0 0 0 0))
   )
-  (wire (pts (xy 72.39 75.565) (xy 69.85 75.565))
-    (stroke (width 0) (type default) (color 0 0 0 0))
-  )
   (wire (pts (xy 74.93 67.945) (xy 69.85 67.945))
     (stroke (width 0) (type default) (color 0 0 0 0))
@@
     (stroke (width 0) (type default) (color 0 0 0 0))
   )
-  (wire (pts (xy 50.165 73.025) (xy 57.15 73.025))
-    (stroke (width 0) (type default) (color 0 0 0 0))
-  )
   (wire (pts (xy 112.395 100.33) (xy 112.395 102.87))
     (stroke (width 0) (type default) (color 0 0 0 0))
@@
     (stroke (width 0) (type default) (color 0 0 0 0))
   )
+  (wire (pts (xy 74.93 73.025) (xy 69.85 73.025))
+    (stroke (width 0) (type default) (color 0 0 0 0))
+  )
   (wire (pts (xy 112.395 95.25) (xy 126.365 95.25))
     (stroke (width 0) (type default) (color 0 0 0 0))
@@
     (stroke (width 0) (type default) (color 0 0 0 0))
   )
-  (wire (pts (xy 69.85 35.56) (xy 83.82 35.56))
-    (stroke (width 0) (type default) (color 0 0 0 0))
-  )
   (wire (pts (xy 153.035 100.33) (xy 153.035 102.87))
     (stroke (width 0) (type default) (color 0 0 0 0))
   )
+  (wire (pts (xy 52.07 73.025) (xy 57.15 73.025))
+    (stroke (width 0) (type default) (color 0 0 0 0))
+  )
   (wire (pts (xy 52.07 33.02) (xy 57.15 33.02))
     (stroke (width 0) (type default) (color 0 0 0 0))
@@
     (stroke (width 0) (type default) (color 0 0 0 0))
   )
-  (global_label "3V3" (shape input) (at 50.165 73.025 180) (fields_autoplaced)
-    (effects (font (size 1.27 1.27)) (justify right))
-    (property "Intersheet References" "${INTERSHEET_REFS}" (id 0) (at 44.2443 73.1044 0)
+  (global_label "3V3" (shape input) (at 52.07 75.565 180) (fields_autoplaced)
+    (effects (font (size 1.27 1.27)) (justify right))
+    (property "Intersheet References" "${INTERSHEET_REFS}" (id 0) (at 46.1493 75.6444 0)
       (effects (font (size 1.27 1.27)) (justify right) hide)
     )
@@
     )
   )
-  (global_label "3V3" (shape input) (at 76.835 73.025 0) (fields_autoplaced)
-    (effects (font (size 1.27 1.27)) (justify left))
-    (property "Intersheet References" "${INTERSHEET_REFS}" (id 0) (at 82.7557 73.1044 0)
-      (effects (font (size 1.27 1.27)) (justify left) hide)
+  (global_label "3V3" (shape input) (at 52.07 73.025 180) (fields_autoplaced)
+    (effects (font (size 1.27 1.27)) (justify right))
+    (property "Intersheet References" "${INTERSHEET_REFS}" (id 0) (at 46.1493 72.9456 0)
+      (effects (font (size 1.27 1.27)) (justify right) hide)
     )
   )
@@
     )
   )
-  (global_label "5V" (shape input) (at 74.93 38.1 0) (fields_autoplaced)
-    (effects (font (size 1.27 1.27)) (justify left))
-    (property "Intersheet References" "${INTERSHEET_REFS}" (id 0) (at 79.6412 38.0206 0)
-      (effects (font (size 1.27 1.27)) (justify left) hide)
-    )
-  )
-  (global_label "5V" (shape input) (at 54.61 75.565 180) (fields_autoplaced)
-    (effects (font (size 1.27 1.27)) (justify right))
-    (property "Intersheet References" "${INTERSHEET_REFS}" (id 0) (at 49.8988 75.4856 0)
+  (global_label "5V" (shape input) (at 52.07 30.48 180) (fields_autoplaced)
+    (effects (font (size 1.27 1.27)) (justify right))
+    (property "Intersheet References" "${INTERSHEET_REFS}" (id 0) (at 47.3588 30.5594 0)
+      (effects (font (size 1.27 1.27)) (justify right) hide)
+    )
+  )
+  (global_label "5V" (shape input) (at 52.07 67.945 180) (fields_autoplaced)
+    (effects (font (size 1.27 1.27)) (justify right))
+    (property "Intersheet References" "${INTERSHEET_REFS}" (id 0) (at 47.3588 67.8656 0)
       (effects (font (size 1.27 1.27)) (justify right) hide)
     )
@@
     )
   )
-  (global_label "5V" (shape input) (at 72.39 75.565 0) (fields_autoplaced)
-    (effects (font (size 1.27 1.27)) (justify left))
-    (property "Intersheet References" "${INTERSHEET_REFS}" (id 0) (at 77.1012 75.4856 0)
-      (effects (font (size 1.27 1.27)) (justify left) hide)
+  (global_label "5V" (shape input) (at 52.07 65.405 180) (fields_autoplaced)
+    (effects (font (size 1.27 1.27)) (justify right))
+    (property "Intersheet References" "${INTERSHEET_REFS}" (id 0) (at 47.3588 65.4844 0)
+      (effects (font (size 1.27 1.27)) (justify right) hide)
     )
   )
@@
     (effects (font (size 1.27 1.27)) (justify right))
   )
-  (hierarchical_label "I2CA_SCL" (shape input) (at 52.07 65.405 180)
-    (effects (font (size 1.27 1.27)) (justify right))
+  (hierarchical_label "I2CA_SCL" (shape input) (at 74.93 73.025 0)
+    (effects (font (size 1.27 1.27)) (justify left))
   )
   (hierarchical_label "SPI_MISO" (shape output) (at 74.93 33.02 0)
     (effects (font (size 1.27 1.27)) (justify left))
   )
-  (hierarchical_label "SPI_SCK" (shape input) (at 52.07 30.48 180)
-    (effects (font (size 1.27 1.27)) (justify right))
-  )
-  (hierarchical_label "I2CA_SDA" (shape bidirectional) (at 52.07 67.945 180)
-    (effects (font (size 1.27 1.27)) (justify right))
+  (hierarchical_label "SPI_SCK" (shape input) (at 74.93 35.56 0)
+    (effects (font (size 1.27 1.27)) (justify left))
+  )
+  (hierarchical_label "I2CA_SDA" (shape bidirectional) (at 74.93 75.565 0)
+    (effects (font (size 1.27 1.27)) (justify left))
   )
   (hierarchical_label "I2CB_SCL" (shape input) (at 74.93 65.405 0)
@@
     (pin "1")
   )
-  (symbol (lib_id "power:GND") (at 83.82 75.565 0) (unit 1)
-    (in_bom yes) (on_board yes) (fields_autoplaced)
-    (property "Reference" "#PWR0170" (id 0) (at 83.82 81.915 0)
-      (effects (font (size 1.27 1.27)) hide)
-    )
-    (property "Value" "GND" (id 1) (at 83.82 80.645 0))
-    (property "Footprint" "" (id 2) (at 83.82 75.565 0)
-      (effects (font (size 1.27 1.27)) hide)
-    )
-    (property "Datasheet" "" (id 3) (at 83.82 75.565 0)
-      (effects (font (size 1.27 1.27)) hide)
-    )
+  (symbol (lib_id "power:GND") (at 86.995 75.565 0) (unit 1)
+    (in_bom yes) (on_board yes) (fields_autoplaced)
+    (property "Reference" "#PWR0170" (id 0) (at 86.995 81.915 0)
+      (effects (font (size 1.27 1.27)) hide)
+    )
+    (property "Value" "GND" (id 1) (at 86.995 80.645 0))
+    (property "Footprint" "" (id 2) (at 86.995 75.565 0)
+      (effects (font (size 1.27 1.27)) hide)
+    )
+    (property "Datasheet" "" (id 3) (at 86.995 75.565 0)
+      (effects (font (size 1.27 1.27)) hide)
+    )

Commit message: continue routing
Connections:
- net 3V3: now also J1003.4 (Pin_4), J1003.8 (Pin_8); no longer J1003.7 (Pin_7), J1003.9 (Pin_9)
- net 5V: now also J1003.7 (Pin_7); no longer J1003.1 (Pin_1)
- net I2CA_SCL: now also J1003.9 (Pin_9); no longer J1003.8 (Pin_8)
- net I2CA_SDA: now also J1003.1 (Pin_1); no longer J1003.10 (Pin_10)
- net I2CB_SCL: now also J1003.10 (Pin_10); no longer J1003.2 (Pin_2)
- net I2CB_SDA: now also J1003.2 (Pin_2); no longer J1003.4 (Pin_4)
- net SPI_CS: now also J1001.4 (Pin_4); no longer J1001.3 (Pin_3)
- net SPI_EOC: now also J1001.2 (Pin_2); no longer J1001.5 (Pin_5)
- net SPI_MISO: now also J1001.6 (Pin_6); no longer J1001.4 (Pin_4)
- net SPI_MOSI: now also J1001.5 (Pin_5); no longer J1001.2 (Pin_2)
- net SPI_SCK: now also J1001.3 (Pin_3); no longer J1001.6 (Pin_6)
Changed lines of the file:
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@@
-    (stroke (width 0) (type default) (color 0 0 0 0))
-  )
-  (wire (pts (xy 43.18 70.485) (xy 43.18 75.565))
     (stroke (width 0) (type default) (color 0 0 0 0))
   )
@@
     (stroke (width 0) (type default) (color 0 0 0 0))
   )
-  (wire (pts (xy 57.15 70.485) (xy 43.18 70.485))
+  (wire (pts (xy 36.83 70.485) (xy 57.15 70.485))
     (stroke (width 0) (type default) (color 0 0 0 0))
   )
@@
     (stroke (width 0) (type default) (color 0 0 0 0))
   )
+  (wire (pts (xy 36.83 75.565) (xy 36.83 70.485))
+    (stroke (width 0) (type default) (color 0 0 0 0))
+  )
   (wire (pts (xy 52.07 73.025) (xy 57.15 73.025))
     (stroke (width 0) (type default) (color 0 0 0 0))
@@
     (stroke (width 0) (type default) (color 0 0 0 0))
   )
-  (global_label "3V3" (shape input) (at 52.07 75.565 180) (fields_autoplaced)
-    (effects (font (size 1.27 1.27)) (justify right))
-    (property "Intersheet References" "${INTERSHEET_REFS}" (id 0) (at 46.1493 75.6444 0)
-      (effects (font (size 1.27 1.27)) (justify right) hide)
+  (global_label "3V3" (shape input) (at 74.93 73.025 0) (fields_autoplaced)
+    (effects (font (size 1.27 1.27)) (justify left))
+    (property "Intersheet References" "${INTERSHEET_REFS}" (id 0) (at 80.8507 72.9456 0)
+      (effects (font (size 1.27 1.27)) (justify left) hide)
     )
   )
@@
     )
   )
-  (global_label "3V3" (shape input) (at 52.07 73.025 180) (fields_autoplaced)
-    (effects (font (size 1.27 1.27)) (justify right))
-    (property "Intersheet References" "${INTERSHEET_REFS}" (id 0) (at 46.1493 72.9456 0)
-      (effects (font (size 1.27 1.27)) (justify right) hide)
+  (global_label "3V3" (shape input) (at 74.93 67.945 0) (fields_autoplaced)
+    (effects (font (size 1.27 1.27)) (justify left))
+    (property "Intersheet References" "${INTERSHEET_REFS}" (id 0) (at 80.8507 68.0244 0)
+      (effects (font (size 1.27 1.27)) (justify left) hide)
     )
   )
@@
     )
   )
-  (global_label "5V" (shape input) (at 52.07 65.405 180) (fields_autoplaced)
-    (effects (font (size 1.27 1.27)) (justify right))
-    (property "Intersheet References" "${INTERSHEET_REFS}" (id 0) (at 47.3588 65.4844 0)
+  (global_label "5V" (shape input) (at 52.07 73.025 180) (fields_autoplaced)
+    (effects (font (size 1.27 1.27)) (justify right))
+    (property "Intersheet References" "${INTERSHEET_REFS}" (id 0) (at 47.3588 73.1044 0)
       (effects (font (size 1.27 1.27)) (justify right) hide)
     )
@@
     (effects (font (size 1.27 1.27)) (justify right))
   )
-  (hierarchical_label "SPI_MOSI" (shape input) (at 74.93 30.48 0)
-    (effects (font (size 1.27 1.27)) (justify left))
-  )
-  (hierarchical_label "SPI_EOC" (shape output) (at 52.07 35.56 180)
-    (effects (font (size 1.27 1.27)) (justify right))
+  (hierarchical_label "SPI_MOSI" (shape input) (at 52.07 35.56 180)
+    (effects (font (size 1.27 1.27)) (justify right))
+  )
+  (hierarchical_label "SPI_EOC" (shape output) (at 74.93 30.48 0)
+    (effects (font (size 1.27 1.27)) (justify left))
   )
   (hierarchical_label "UARTC_TX" (shape input) (at 121.285 59.055 180)
@@
     (effects (font (size 1.27 1.27)) (justify left))
   )
-  (hierarchical_label "SPI_CS" (shape input) (at 52.07 33.02 180)
-    (effects (font (size 1.27 1.27)) (justify right))
-  )
-  (hierarchical_label "I2CB_SDA" (shape bidirectional) (at 74.93 67.945 0)
+  (hierarchical_label "SPI_CS" (shape input) (at 74.93 33.02 0)
+    (effects (font (size 1.27 1.27)) (justify left))
+  )
+  (hierarchical_label "I2CB_SDA" (shape bidirectional) (at 74.93 65.405 0)
     (effects (font (size 1.27 1.27)) (justify left))
   )
@@
     (effects (font (size 1.27 1.27)) (justify right))
   )
-  (hierarchical_label "I2CA_SCL" (shape input) (at 74.93 73.025 0)
-    (effects (font (size 1.27 1.27)) (justify left))
-  )
-  (hierarchical_label "SPI_MISO" (shape output) (at 74.93 33.02 0)
-    (effects (font (size 1.27 1.27)) (justify left))
-  )
-  (hierarchical_label "SPI_SCK" (shape input) (at 74.93 35.56 0)
-    (effects (font (size 1.27 1.27)) (justify left))
-  )
-  (hierarchical_label "I2CA_SDA" (shape bidirectional) (at 74.93 75.565 0)
-    (effects (font (size 1.27 1.27)) (justify left))
-  )
-  (hierarchical_label "I2CB_SCL" (shape input) (at 74.93 65.405 0)
+  (hierarchical_label "I2CA_SCL" (shape input) (at 52.07 75.565 180)
+    (effects (font (size 1.27 1.27)) (justify right))
+  )
+  (hierarchical_label "SPI_MISO" (shape output) (at 74.93 35.56 0)
+    (effects (font (size 1.27 1.27)) (justify left))
+  )
+  (hierarchical_label "SPI_SCK" (shape input) (at 52.07 33.02 180)
+    (effects (font (size 1.27 1.27)) (justify right))
+  )
+  (hierarchical_label "I2CA_SDA" (shape bidirectional) (at 52.07 65.405 180)
+    (effects (font (size 1.27 1.27)) (justify right))
+  )
+  (hierarchical_label "I2CB_SCL" (shape input) (at 74.93 75.565 0)
     (effects (font (size 1.27 1.27)) (justify left))
   )
@@
     (pin "1")
   )
-  (symbol (lib_id "power:GND") (at 43.18 75.565 0) (mirror y) (unit 1)
-    (in_bom yes) (on_board yes) (fields_autoplaced)
-    (property "Reference" "#PWR0171" (id 0) (at 43.18 81.915 0)
-      (effects (font (size 1.27 1.27)) hide)
-    )
-    (property "Value" "GND" (id 1) (at 43.18 80.645 0))
-    (property "Footprint" "" (id 2) (at 43.18 75.565 0)
-      (effects (font (size 1.27 1.27)) hide)
-    )
-    (property "Datasheet" "" (id 3) (at 43.18 75.565 0)
-      (effects (font (size 1.27 1.27)) hide)
-    )
+  (symbol (lib_id "power:GND") (at 36.83 75.565 0) (mirror y) (unit 1)
+    (in_bom yes) (on_board yes) (fields_autoplaced)
+    (property "Reference" "#PWR0171" (id 0) (at 36.83 81.915 0)
+      (effects (font (size 1.27 1.27)) hide)
+    )
+    (property "Value" "GND" (id 1) (at 36.83 80.645 0))
+    (property "Footprint" "" (id 2) (at 36.83 75.565 0)
+      (effects (font (size 1.27 1.27)) hide)
+    )
+    (property "Datasheet" "" (id 3) (at 36.83 75.565 0)
+      (effects (font (size 1.27 1.27)) hide)
+    )

Commit message: routing: connected everything
Parts:
- removed J1002, J1004: UART externa x2, Connector_PinHeader_2.54mm:PinHeader_2x04_P2.54mm_Horizontal, symbol Connector_Generic:Conn_02x04_Odd_Even
- added J1: Conn_02x06_Odd_Even, Connector_PinHeader_2.54mm:PinHeader_2x06_P2.54mm_Horizontal, symbol Connector_Generic:Conn_02x06_Odd_Even
Connections:
- net 3V3: now also J1.10 (Pin_10), J1.2 (Pin_2), J1.6 (Pin_6)
- net GND: now also J1.12 (Pin_12), J1.4 (Pin_4), J1.8 (Pin_8)
- net I2CA_SCL: now also J1003.1 (Pin_1); no longer J1003.9 (Pin_9)
- net I2CA_SDA: now also J1003.9 (Pin_9); no longer J1003.1 (Pin_1)
- net I2CB_SCL: now also J1003.2 (Pin_2); no longer J1003.10 (Pin_10)
- net I2CB_SDA: now also J1003.10 (Pin_10); no longer J1003.2 (Pin_2)
- net UARTA_RX: now also J1.5 (Pin_5)
- net UARTA_TX: now also J1.7 (Pin_7)
- net UARTB_RX: now also J1.1 (Pin_1)
- net UARTB_TX: now also J1.3 (Pin_3)
- net UARTC_RX: now also J1.9 (Pin_9)
- net UARTC_TX: now also J1.11 (Pin_11)
