File: hardware/Drone FCC/conexiones_extra.kicad_sch (KiCad schematic)
At the start: 4 parts, among them J1 Conn_02x06_Odd_Even, J1001 SPI externo, J1003 I2C externo x2, J1005 5V y 3V3 x 2

Commit message: positioned components in 100x60 board with incomplete routing
Parts:
- J1: value Conn_02x06_Odd_Even -> UARTs externo x 3
Connections:
- net 3V3: now also J1.11 (Pin_11), J1.3 (Pin_3), J1.7 (Pin_7), J1001.2 (Pin_2), J1003.2 (Pin_2); no longer J1.10 (Pin_10), J1.2 (Pin_2), J1.6 (Pin_6), J1001.7 (Pin_7), J1003.8 (Pin_8)
- net 5V: now also J1003.1 (Pin_1); no longer J1003.7 (Pin_7)
- net GND: now also J1001.4 (Pin_4); no longer J1001.8 (Pin_8)
- net I2CA_SCL: now also J1003.9 (Pin_9); no longer J1003.1 (Pin_1)
- net I2CA_SDA: now also J1003.7 (Pin_7); no longer J1003.9 (Pin_9)
- net I2CB_SCL: now also J1003.10 (Pin_10); no longer J1003.2 (Pin_2)
- net I2CB_SDA: now also J1003.8 (Pin_8); no longer J1003.10 (Pin_10)
- net SPI_CS: now also J1001.5 (Pin_5); no longer J1001.4 (Pin_4)
- net SPI_EOC: now also J1001.3 (Pin_3); no longer J1001.2 (Pin_2)
- net SPI_MISO: now also J1001.7 (Pin_7); no longer J1001.6 (Pin_6)
- net SPI_MOSI: now also J1001.8 (Pin_8); no longer J1001.5 (Pin_5)
- net SPI_SCK: now also J1001.6 (Pin_6); no longer J1001.3 (Pin_3)
- net UARTA_RX: now also J1.9 (Pin_9); no longer J1.5 (Pin_5)
- net UARTA_TX: now also J1.10 (Pin_10); no longer J1.7 (Pin_7)
- net UARTB_RX: now also J1.5 (Pin_5); no longer J1.1 (Pin_1)
- net UARTB_TX: now also J1.6 (Pin_6); no longer J1.3 (Pin_3)
- net UARTC_RX: now also J1.1 (Pin_1); no longer J1.9 (Pin_9)
- net UARTC_TX: now also J1.2 (Pin_2); no longer J1.11 (Pin_11)
Other:
- moved on the sheet: J1

Commit message: todo: route SWD connector
Connections:
- net 3V3: now also J1003.10 (Pin_10), J1003.8 (Pin_8); no longer J1003.2 (Pin_2), J1003.4 (Pin_4)
- net 5V: now also J1003.7 (Pin_7), J1003.9 (Pin_9); no longer J1003.1 (Pin_1), J1003.3 (Pin_3)
- net I2CA_SCL: now also J1003.3 (Pin_3); no longer J1003.9 (Pin_9)
- net I2CA_SDA: now also J1003.1 (Pin_1); no longer J1003.7 (Pin_7)
- net I2CB_SCL: now also J1003.4 (Pin_4); no longer J1003.10 (Pin_10)
- net I2CB_SDA: now also J1003.2 (Pin_2); no longer J1003.8 (Pin_8)
Changed lines of the file:
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@@
     (stroke (width 0) (type default) (color 0 0 0 0))
   )
-  (wire (pts (xy 74.93 73.025) (xy 69.85 73.025))
-    (stroke (width 0) (type default) (color 0 0 0 0))
-  )
-  (wire (pts (xy 49.53 67.945) (xy 57.15 67.945))
+  (wire (pts (xy 74.93 65.405) (xy 69.85 65.405))
+    (stroke (width 0) (type default) (color 0 0 0 0))
+  )
+  (wire (pts (xy 49.53 75.565) (xy 57.15 75.565))
     (stroke (width 0) (type default) (color 0 0 0 0))
   )
@@
     (stroke (width 0) (type default) (color 0 0 0 0))
   )
-  (wire (pts (xy 52.07 75.565) (xy 57.15 75.565))
+  (wire (pts (xy 52.07 67.945) (xy 57.15 67.945))
     (stroke (width 0) (type default) (color 0 0 0 0))
   )
@@
     (stroke (width 0) (type default) (color 0 0 0 0))
   )
-  (wire (pts (xy 52.07 73.025) (xy 57.15 73.025))
+  (wire (pts (xy 52.07 65.405) (xy 57.15 65.405))
     (stroke (width 0) (type default) (color 0 0 0 0))
   )
@@
     (stroke (width 0) (type default) (color 0 0 0 0))
   )
-  (wire (pts (xy 54.61 65.405) (xy 57.15 65.405))
+  (wire (pts (xy 54.61 73.025) (xy 57.15 73.025))
     (stroke (width 0) (type default) (color 0 0 0 0))
   )
@@
     (stroke (width 0) (type default) (color 0 0 0 0))
   )
-  (wire (pts (xy 69.85 65.405) (xy 72.39 65.405))
+  (wire (pts (xy 69.85 73.025) (xy 72.39 73.025))
     (stroke (width 0) (type default) (color 0 0 0 0))
   )
@@
     (stroke (width 0) (type default) (color 0 0 0 0))
   )
-  (wire (pts (xy 69.85 67.945) (xy 78.74 67.945))
+  (wire (pts (xy 69.85 75.565) (xy 78.74 75.565))
     (stroke (width 0) (type default) (color 0 0 0 0))
   )
@@
     (stroke (width 0) (type default) (color 0 0 0 0))
   )
-  (wire (pts (xy 69.85 75.565) (xy 74.93 75.565))
+  (wire (pts (xy 69.85 67.945) (xy 74.93 67.945))
     (stroke (width 0) (type default) (color 0 0 0 0))
   )
@@
     (stroke (width 0) (type default) (color 0 0 0 0))
   )
-  (global_label "3V3" (shape input) (at 72.39 65.405 0) (fields_autoplaced)
-    (effects (font (size 1.27 1.27)) (justify left))
-    (property "Intersheet References" "${INTERSHEET_REFS}" (id 0) (at 78.3107 65.3256 0)
+  (global_label "3V3" (shape input) (at 72.39 73.025 0) (fields_autoplaced)
+    (effects (font (size 1.27 1.27)) (justify left))
+    (property "Intersheet References" "${INTERSHEET_REFS}" (id 0) (at 78.3107 72.9456 0)
       (effects (font (size 1.27 1.27)) (justify left) hide)
     )
@@
     )
   )
-  (global_label "3V3" (shape input) (at 78.74 67.945 0) (fields_autoplaced)
-    (effects (font (size 1.27 1.27)) (justify left))
-    (property "Intersheet References" "${INTERSHEET_REFS}" (id 0) (at 84.6607 68.0244 0)
+  (global_label "3V3" (shape input) (at 78.74 75.565 0) (fields_autoplaced)
+    (effects (font (size 1.27 1.27)) (justify left))
+    (property "Intersheet References" "${INTERSHEET_REFS}" (id 0) (at 84.6607 75.6444 0)
       (effects (font (size 1.27 1.27)) (justify left) hide)
     )
@@
     )
   )
-  (global_label "5V" (shape input) (at 49.53 67.945 180) (fields_autoplaced)
-    (effects (font (size 1.27 1.27)) (justify right))
-    (property "Intersheet References" "${INTERSHEET_REFS}" (id 0) (at 44.8188 67.8656 0)
+  (global_label "5V" (shape input) (at 49.53 75.565 180) (fields_autoplaced)
+    (effects (font (size 1.27 1.27)) (justify right))
+    (property "Intersheet References" "${INTERSHEET_REFS}" (id 0) (at 44.8188 75.4856 0)
       (effects (font (size 1.27 1.27)) (justify right) hide)
     )
@@
     )
   )
-  (global_label "5V" (shape input) (at 54.61 65.405 180) (fields_autoplaced)
-    (effects (font (size 1.27 1.27)) (justify right))
-    (property "Intersheet References" "${INTERSHEET_REFS}" (id 0) (at 49.8988 65.4844 0)
+  (global_label "5V" (shape input) (at 54.61 73.025 180) (fields_autoplaced)
+    (effects (font (size 1.27 1.27)) (justify right))
+    (property "Intersheet References" "${INTERSHEET_REFS}" (id 0) (at 49.8988 73.1044 0)
       (effects (font (size 1.27 1.27)) (justify right) hide)
     )
@@
     (effects (font (size 1.27 1.27)) (justify right))
   )
-  (hierarchical_label "I2CB_SDA" (shape bidirectional) (at 74.93 73.025 0)
+  (hierarchical_label "I2CB_SDA" (shape bidirectional) (at 74.93 65.405 0)
     (effects (font (size 1.27 1.27)) (justify left))
   )
@@
     (effects (font (size 1.27 1.27)) (justify left))
   )
-  (hierarchical_label "I2CA_SCL" (shape input) (at 52.07 75.565 180)
+  (hierarchical_label "I2CA_SCL" (shape input) (at 52.07 67.945 180)
     (effects (font (size 1.27 1.27)) (justify right))
   )
@@
     (effects (font (size 1.27 1.27)) (justify left))
   )
-  (hierarchical_label "I2CA_SDA" (shape bidirectional) (at 52.07 73.025 180)
-    (effects (font (size 1.27 1.27)) (justify right))
-  )
-  (hierarchical_label "I2CB_SCL" (shape input) (at 74.93 75.565 0)
-    (effects (font (size 1.27 1.27)) (justify left))
-  )
+  (hierarchical_label "I2CA_SDA" (shape bidirectional) (at 52.07 65.405 180)
+    (effects (font (size 1.27 1.27)) (justify right))
+  )
+  (hierarchical_label "I2CB_SCL" (shape input) (at 74.93 67.945 0)
+    (effects (font (size 1.27 1.27)) (justify left))
+  )

Commit message: added LEDs in routing
Connections:
- net SPI_MISO: now also J1001.8 (Pin_8); no longer J1001.7 (Pin_7)
- net SPI_MOSI: now also J1001.7 (Pin_7); no longer J1001.8 (Pin_8)
Changed lines of the file:
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@@
     (effects (font (size 1.27 1.27)) (justify right))
   )
-  (hierarchical_label "SPI_MOSI" (shape input) (at 74.93 38.1 0)
-    (effects (font (size 1.27 1.27)) (justify left))
+  (hierarchical_label "SPI_MOSI" (shape input) (at 52.07 38.1 180)
+    (effects (font (size 1.27 1.27)) (justify right))
   )
   (hierarchical_label "SPI_EOC" (shape output) (at 52.07 33.02 180)
@@
     (effects (font (size 1.27 1.27)) (justify right))
   )
-  (hierarchical_label "SPI_MISO" (shape output) (at 52.07 38.1 180)
-    (effects (font (size 1.27 1.27)) (justify right))
+  (hierarchical_label "SPI_MISO" (shape output) (at 74.93 38.1 0)
+    (effects (font (size 1.27 1.27)) (justify left))
   )
   (hierarchical_label "SPI_SCK" (shape input) (at 74.93 35.56 0)

Commit message: finished
Connections:
- net GND: now also J1.1 (Pin_1), J1.5 (Pin_5), J1.9 (Pin_9), J1001.7 (Pin_7), J1003.3 (Pin_3), J1003.4 (Pin_4); no longer J1.12 (Pin_12), J1.4 (Pin_4), J1.8 (Pin_8), J1001.4 (Pin_4), J1003.5 (Pin_5), J1003.6 (Pin_6)
- net I2CA_SCL: now also J1003.5 (Pin_5); no longer J1003.3 (Pin_3)
- net I2CB_SCL: now also J1003.6 (Pin_6); no longer J1003.4 (Pin_4)
- net SPI_CS: now also J1001.4 (Pin_4); no longer J1001.5 (Pin_5)
- net SPI_EOC: now also J1001.6 (Pin_6); no longer J1001.3 (Pin_3)
- net SPI_MISO: now also J1001.5 (Pin_5); no longer J1001.8 (Pin_8)
- net SPI_MOSI: now also J1001.3 (Pin_3); no longer J1001.7 (Pin_7)
- net SPI_SCK: now also J1001.8 (Pin_8); no longer J1001.6 (Pin_6)
- net UARTA_RX: now also J1.12 (Pin_12); no longer J1.9 (Pin_9)
- net UARTB_RX: now also J1.8 (Pin_8); no longer J1.5 (Pin_5)
- net UARTC_RX: now also J1.4 (Pin_4); no longer J1.1 (Pin_1)
