File: hardware/Drone FCC/debug.kicad_sch (KiCad schematic)
At the start: 6 parts, among them J601 SWD Debug Connector

Commit message: removed all the TVS from the PCB and SCH
Parts:
- removed D601, D602, D603, D604, D605: D_TVS, Diode_SMD:D_0402_1005Metric_Pad0.77x0.64mm_HandSolder, symbol Device:D_TVS
Changed lines of the file:
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@@
     (pin "1")
-  )
-  (symbol (lib_id "Device:D_TVS") (at 169.545 93.345 90) (unit 1)
-    (in_bom yes) (on_board yes)
-    (property "Reference" "D605" (id 0) (at 175.895 100.33 0)
-      (effects (font (size 1.27 1.27)) (justify left))
-    )
-    (property "Value" "D_TVS" (id 1) (at 173.355 100.33 0)
-      (effects (font (size 1.27 1.27)) (justify left))
-    )
-    (property "Footprint" "Diode_SMD:D_0402_1005Metric_Pad0.77x0.64mm_HandSolder" (id 2) (at 169.545 93.345 0)
-      (effects (font (size 1.27 1.27)) hide)
-    )
-    (property "Datasheet" "~" (id 3) (at 169.545 93.345 0)
-      (effects (font (size 1.27 1.27)) hide)
-    )
-    (pin "1")
-    (pin "2")
-  )
-  (symbol (lib_id "Device:D_TVS") (at 150.495 93.345 90) (unit 1)
-    (in_bom yes) (on_board yes)
-    (property "Reference" "D603" (id 0) (at 156.845 100.33 0)
-      (effects (font (size 1.27 1.27)) (justify left))
-    )
-    (property "Value" "D_TVS" (id 1) (at 154.305 100.33 0)
-      (effects (font (size 1.27 1.27)) (justify left))
-    )
-    (property "Footprint" "Diode_SMD:D_0402_1005Metric_Pad0.77x0.64mm_HandSolder" (id 2) (at 150.495 93.345 0)
-      (effects (font (size 1.27 1.27)) hide)
-    )
-    (property "Datasheet" "~" (id 3) (at 150.495 93.345 0)
-      (effects (font (size 1.27 1.27)) hide)
-    )
-    (pin "1")
-    (pin "2")
   )
   (symbol (lib_id "power:GND") (at 140.97 99.06 0) (mirror y) (unit 1)
@@
     (pin "6")
   )
-  (symbol (lib_id "Device:D_TVS") (at 160.02 93.345 90) (unit 1)
-    (in_bom yes) (on_board yes)
-    (property "Reference" "D604" (id 0) (at 166.37 100.33 0)
-      (effects (font (size 1.27 1.27)) (justify left))
-    )
-    (property "Value" "D_TVS" (id 1) (at 163.83 100.33 0)
-      (effects (font (size 1.27 1.27)) (justify left))
-    )
-    (property "Footprint" "Diode_SMD:D_0402_1005Metric_Pad0.77x0.64mm_HandSolder" (id 2) (at 160.02 93.345 0)
-      (effects (font (size 1.27 1.27)) hide)
-    )
-    (property "Datasheet" "~" (id 3) (at 160.02 93.345 0)
-      (effects (font (size 1.27 1.27)) hide)
-    )
-    (pin "1")
-    (pin "2")
-  )
-  (symbol (lib_id "Device:D_TVS") (at 131.445 93.345 90) (unit 1)
-    (in_bom yes) (on_board yes)
-    (property "Reference" "D601" (id 0) (at 137.795 100.33 0)
-      (effects (font (size 1.27 1.27)) (justify left))
-    )
-    (property "Value" "D_TVS" (id 1) (at 135.255 100.33 0)
-      (effects (font (size 1.27 1.27)) (justify left))
-    )
-    (property "Footprint" "Diode_SMD:D_0402_1005Metric_Pad0.77x0.64mm_HandSolder" (id 2) (at 131.445 93.345 0)
-      (effects (font (size 1.27 1.27)) hide)
-    )
-    (property "Datasheet" "~" (id 3) (at 131.445 93.345 0)
-      (effects (font (size 1.27 1.27)) hide)
-    )
-    (pin "1")
-    (pin "2")
-  )
-  (symbol (lib_id "Device:D_TVS") (at 140.97 93.345 90) (unit 1)
-    (in_bom yes) (on_board yes)
-    (property "Reference" "D602" (id 0) (at 147.32 100.33 0)
-      (effects (font (size 1.27 1.27)) (justify left))
-    )
-    (property "Value" "D_TVS" (id 1) (at 144.78 100.33 0)
-      (effects (font (size 1.27 1.27)) (justify left))
-    )
-    (property "Footprint" "Diode_SMD:D_0402_1005Metric_Pad0.77x0.64mm_HandSolder" (id 2) (at 140.97 93.345 0)
-      (effects (font (size 1.27 1.27)) hide)
-    )
-    (property "Datasheet" "~" (id 3) (at 140.97 93.345 0)
-      (effects (font (size 1.27 1.27)) hide)
-    )
-    (pin "1")
-    (pin "2")
-  )
   (symbol (lib_id "power:GND") (at 150.495 99.06 0) (mirror y) (unit 1)
