File: hardware/Drone FCC/motores_servos_pwm.kicad_sch (KiCad schematic)
At the start: 14 parts, among them J301 ESC 1, J302 ESC 2, J303 ESC 3, J304 ESC 4, J305 ESC 5, J306 ESC 6, J307 ESC 7, J308 ESC 8, J309 SERVO 1, J310 SERVO 2, J311 SERVO 3, J312 SERVO 4, J313 Power Servo

Commit message: re enumeation of componentes
Parts:
- renumbered J313 to J10, J309 to J11, J310 to J12, J311 to J13, J312 to J14, J301 to J2, J302 to J3, J303 to J4, J304 to J5, J305 to J6, J306 to J7, J307 to J8, J308 to J9, JP301 to JP1
Changed lines of the file:
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@@
   (symbol (lib_id "Connector_Generic:Conn_01x03") (at 201.295 84.455 0) (mirror y) (unit 1)
     (in_bom yes) (on_board yes) (fields_autoplaced)
-    (property "Reference" "J311" (id 0) (at 201.295 74.93 0))
+    (property "Reference" "J13" (id 0) (at 201.295 74.93 0))
     (property "Value" "SERVO 3" (id 1) (at 201.295 77.47 0))
     (property "Footprint" "TSW-101-08-G-T-RA:SAMTEC_TSW-101-08-G-T-RA" (id 2) (at 201.295 84.455 0)
@@
   (symbol (lib_id "Connector_Generic:Conn_01x03") (at 68.58 116.205 0) (mirror y) (unit 1)
     (in_bom yes) (on_board yes) (fields_autoplaced)
-    (property "Reference" "J305" (id 0) (at 68.58 106.68 0))
+    (property "Reference" "J6" (id 0) (at 68.58 106.68 0))
     (property "Value" "ESC 5" (id 1) (at 68.58 109.22 0))
     (property "Footprint" "TSW-101-08-G-T-RA:SAMTEC_TSW-101-08-G-T-RA" (id 2) (at 68.58 116.205 0)
@@
   (symbol (lib_id "power:GND") (at 212.725 69.85 0) (unit 1)
     (in_bom yes) (on_board yes) (fields_autoplaced)
-    (property "Reference" "#PWR019" (id 0) (at 212.725 76.2 0)
+    (property "Reference" "#PWR016" (id 0) (at 212.725 76.2 0)
       (effects (font (size 1.27 1.27)) hide)
     )
@@
   (symbol (lib_id "power:GND") (at 80.01 160.655 0) (unit 1)
     (in_bom yes) (on_board yes) (fields_autoplaced)
-    (property "Reference" "#PWR016" (id 0) (at 80.01 167.005 0)
+    (property "Reference" "#PWR012" (id 0) (at 80.01 167.005 0)
       (effects (font (size 1.27 1.27)) hide)
     )
@@
   (symbol (lib_id "Connector_Generic:Conn_01x03") (at 68.58 34.29 0) (mirror y) (unit 1)
     (in_bom yes) (on_board yes) (fields_autoplaced)
-    (property "Reference" "J301" (id 0) (at 68.58 24.765 0))
+    (property "Reference" "J2" (id 0) (at 68.58 24.765 0))
     (property "Value" "ESC 1" (id 1) (at 68.58 27.305 0))
     (property "Footprint" "TSW-101-08-G-T-RA:SAMTEC_TSW-101-08-G-T-RA" (id 2) (at 68.58 34.29 0)
@@
   (symbol (lib_id "power:GND") (at 80.01 57.785 0) (unit 1)
     (in_bom yes) (on_board yes) (fields_autoplaced)
-    (property "Reference" "#PWR011" (id 0) (at 80.01 64.135 0)
+    (property "Reference" "#PWR07" (id 0) (at 80.01 64.135 0)
       (effects (font (size 1.27 1.27)) hide)
     )
@@
   (symbol (lib_id "power:GND") (at 80.01 140.335 0) (unit 1)
     (in_bom yes) (on_board yes) (fields_autoplaced)
-    (property "Reference" "#PWR015" (id 0) (at 80.01 146.685 0)
+    (property "Reference" "#PWR011" (id 0) (at 80.01 146.685 0)
       (effects (font (size 1.27 1.27)) hide)
     )
@@
   (symbol (lib_id "Connector_Generic:Conn_01x03") (at 68.58 53.34 0) (mirror y) (unit 1)
     (in_bom yes) (on_board yes) (fields_autoplaced)
-    (property "Reference" "J302" (id 0) (at 68.58 43.815 0))
+    (property "Reference" "J3" (id 0) (at 68.58 43.815 0))
     (property "Value" "ESC 2" (id 1) (at 68.58 46.355 0))
     (property "Footprint" "TSW-101-08-G-T-RA:SAMTEC_TSW-101-08-G-T-RA" (id 2) (at 68.58 53.34 0)
@@
   (symbol (lib_id "Connector_Generic:Conn_01x03") (at 201.295 103.505 0) (mirror y) (unit 1)
     (in_bom yes) (on_board yes) (fields_autoplaced)
-    (property "Reference" "J312" (id 0) (at 201.295 93.98 0))
+    (property "Reference" "J14" (id 0) (at 201.295 93.98 0))
     (property "Value" "SERVO 4" (id 1) (at 201.295 96.52 0))
     (property "Footprint" "TSW-101-08-G-T-RA:SAMTEC_TSW-101-08-G-T-RA" (id 2) (at 201.295 103.505 0)
@@
   (symbol (lib_id "Connector_Generic:Conn_01x03") (at 68.58 73.025 0) (mirror y) (unit 1)
     (in_bom yes) (on_board yes)
-    (property "Reference" "J303" (id 0) (at 68.58 59.69 0))
+    (property "Reference" "J4" (id 0) (at 68.58 59.69 0))
     (property "Value" "ESC 3" (id 1) (at 68.58 62.23 0))
     (property "Footprint" "TSW-101-08-G-T-RA:SAMTEC_TSW-101-08-G-T-RA" (id 2) (at 68.58 73.025 0)
@@
   (symbol (lib_id "power:GND") (at 80.01 101.6 0) (unit 1)
     (in_bom yes) (on_board yes) (fields_autoplaced)
-    (property "Reference" "#PWR013" (id 0) (at 80.01 107.95 0)
+    (property "Reference" "#PWR09" (id 0) (at 80.01 107.95 0)
       (effects (font (size 1.27 1.27)) hide)
     )
@@
   (symbol (lib_id "Connector_Generic:Conn_01x03") (at 201.295 46.355 0) (mirror y) (unit 1)
     (in_bom yes) (on_board yes)
-    (property "Reference" "J309" (id 0) (at 201.295 36.83 0))
+    (property "Reference" "J11" (id 0) (at 201.295 36.83 0))
     (property "Value" "SERVO 1" (id 1) (at 201.295 39.37 0))
     (property "Footprint" "TSW-101-08-G-T-RA:SAMTEC_TSW-101-08-G-T-RA" (id 2) (at 201.295 46.355 0)
@@
   (symbol (lib_id "power:GND") (at 212.725 50.8 0) (unit 1)
     (in_bom yes) (on_board yes) (fields_autoplaced)
-    (property "Reference" "#PWR018" (id 0) (at 212.725 57.15 0)
+    (property "Reference" "#PWR015" (id 0) (at 212.725 57.15 0)
       (effects (font (size 1.27 1.27)) hide)
     )
@@
   (symbol (lib_id "power:GND") (at 212.725 107.95 0) (unit 1)
     (in_bom yes) (on_board yes) (fields_autoplaced)
-    (property "Reference" "#PWR021" (id 0) (at 212.725 114.3 0)
+    (property "Reference" "#PWR018" (id 0) (at 212.725 114.3 0)
       (effects (font (size 1.27 1.27)) hide)
     )
@@
   (symbol (lib_id "Connector_Generic:Conn_01x03") (at 68.58 97.155 0) (mirror y) (unit 1)
     (in_bom yes) (on_board yes) (fields_autoplaced)
-    (property "Reference" "J304" (id 0) (at 68.58 87.63 0))
+    (property "Reference" "J5" (id 0) (at 68.58 87.63 0))
     (property "Value" "ESC 4" (id 1) (at 68.58 90.17 0))
     (property "Footprint" "TSW-101-08-G-T-RA:SAMTEC_TSW-101-08-G-T-RA" (id 2) (at 68.58 97.155 0)
@@
   (symbol (lib_id "power:GND") (at 80.01 77.47 0) (unit 1)
     (in_bom yes) (on_board yes) (fields_autoplaced)
-    (property "Reference" "#PWR012" (id 0) (at 80.01 83.82 0)
+    (property "Reference" "#PWR08" (id 0) (at 80.01 83.82 0)
       (effects (font (size 1.27 1.27)) hide)
     )
@@
   (symbol (lib_id "power:GND") (at 212.725 88.9 0) (unit 1)
     (in_bom yes) (on_board yes) (fields_autoplaced)
-    (property "Reference" "#PWR020" (id 0) (at 212.725 95.25 0)
+    (property "Reference" "#PWR017" (id 0) (at 212.725 95.25 0)
       (effects (font (size 1.27 1.27)) hide)
     )
@@
   (symbol (lib_id "Connector_Generic:Conn_01x03") (at 68.58 175.895 0) (mirror y) (unit 1)
     (in_bom yes) (on_board yes)
-    (property "Reference" "J308" (id 0) (at 68.58 166.37 0))
+    (property "Reference" "J9" (id 0) (at 68.58 166.37 0))
     (property "Value" "ESC 8" (id 1) (at 68.58 168.91 0))
     (property "Footprint" "TSW-101-08-G-T-RA:SAMTEC_TSW-101-08-G-T-RA" (id 2) (at 68.58 175.895 0)
@@
   (symbol (lib_id "Connector_Generic:Conn_01x02") (at 165.1 25.4 0) (unit 1)
     (in_bom yes) (on_board yes) (fields_autoplaced)
-    (property "Reference" "J313" (id 0) (at 167.64 25.3999 0)
+    (property "Reference" "J10" (id 0) (at 167.64 25.3999 0)
       (effects (font (size 1.27 1.27)) (justify left))
     )
@@
   (symbol (lib_id "Jumper:SolderJumper_2_Open") (at 161.925 64.135 0) (unit 1)
     (in_bom yes) (on_board yes) (fields_autoplaced)
-    (property "Reference" "JP301" (id 0) (at 161.925 58.42 0))
+    (property "Reference" "JP1" (id 0) (at 161.925 58.42 0))
     (property "Value" "SolderJumper_2_Open" (id 1) (at 161.925 60.96 0))
     (property "Footprint" "Jumper:SolderJumper-2_P1.3mm_Open_Pad1.0x1.5mm" (id 2) (at 161.925 64.135 0)
@@
   (symbol (lib_id "Connector_Generic:Conn_01x03") (at 68.58 156.21 0) (mirror y) (unit 1)
     (in_bom yes) (on_board yes)
-    (property "Reference" "J307" (id 0) (at 68.58 147.955 0))
+    (property "Reference" "J8" (id 0) (at 68.58 147.955 0))
     (property "Value" "ESC 7" (id 1) (at 68.58 150.495 0))
     (property "Footprint" "TSW-101-08-G-T-RA:SAMTEC_TSW-101-08-G-T-RA" (id 2) (at 68.58 156.21 0)
@@
   (symbol (lib_id "power:GND") (at 80.01 180.34 0) (unit 1)
     (in_bom yes) (on_board yes) (fields_autoplaced)
-    (property "Reference" "#PWR017" (id 0) (at 80.01 186.69 0)
+    (property "Reference" "#PWR013" (id 0) (at 80.01 186.69 0)
       (effects (font (size 1.27 1.27)) hide)
     )
@@
   (symbol (lib_id "power:GND") (at 80.01 120.65 0) (unit 1)
     (in_bom yes) (on_board yes) (fields_autoplaced)
-    (property "Reference" "#PWR014" (id 0) (at 80.01 127 0)
+    (property "Reference" "#PWR010" (id 0) (at 80.01 127 0)
       (effects (font (size 1.27 1.27)) hide)
     )
@@
   (symbol (lib_id "Connector_Generic:Conn_01x03") (at 68.58 135.89 0) (mirror y) (unit 1)
     (in_bom yes) (on_board yes)
-    (property "Reference" "J306" (id 0) (at 68.58 127 0))
+    (property "Reference" "J7" (id 0) (at 68.58 127 0))
     (property "Value" "ESC 6" (id 1) (at 68.58 128.905 0))
     (property "Footprint" "TSW-101-08-G-T-RA:SAMTEC_TSW-101-08-G-T-RA" (id 2) (at 68.58 135.89 0)
@@
   (symbol (lib_id "Connector_Generic:Conn_01x03") (at 201.295 65.405 0) (mirror y) (unit 1)
     (in_bom yes) (on_board yes) (fields_autoplaced)
-    (property "Reference" "J310" (id 0) (at 201.295 55.88 0))
+    (property "Reference" "J12" (id 0) (at 201.295 55.88 0))
     (property "Value" "SERVO 2" (id 1) (at 201.295 58.42 0))
     (property "Footprint" "TSW-101-08-G-T-RA:SAMTEC_TSW-101-08-G-T-RA" (id 2) (at 201.295 65.405 0)
@@
   (symbol (lib_id "power:GND") (at 157.48 31.75 0) (unit 1)
     (in_bom yes) (on_board yes) (fields_autoplaced)
-    (property "Reference" "#PWR0163" (id 0) (at 157.48 38.1 0)
+    (property "Reference" "#PWR014" (id 0) (at 157.48 38.1 0)
       (effects (font (size 1.27 1.27)) hide)
     )
@@
   (symbol (lib_id "power:GND") (at 80.01 38.735 0) (unit 1)
     (in_bom yes) (on_board yes) (fields_autoplaced)
-    (property "Reference" "#PWR010" (id 0) (at 80.01 45.085 0)
-      (effects (font (size 1.27 1.27)) hide)
-    )
+    (property "Reference" "#PWR06" (id 0) (at 80.01 45.085 0)
+      (effects (font (size 1.27 1.27)) hide)
+    )
