File: hardware/Power switch test/Power switch test.kicad_sch (KiCad schematic)
At the start: 14 parts, among them J1 Vin, J2 Vout, Q1 IRF7425, U1 LD1117S33TR_SOT223

Commit message: start routing
Parts:
- removed Q1: IRF7425, Package_SO:SO-8_3.9x4.9mm_P1.27mm, symbol Device:Q_PMOS_GSD
- removed U1: LD1117S33TR_SOT223, Package_TO_SOT_SMD:SOT-223-3_TabPin2, symbol Regulator_Linear:LD1117S33TR_SOT223
- added Q1: AO3401A, Package_TO_SOT_SMD:SOT-23, symbol Transistor_FET:AO3401A
- added U1: LM1117-3.3, symbol Regulator_Linear:LM1117-3.3
- D1, D2: value 1N5822 -> SS210
Connections:
- net 3V3: now also U1.2 (VO)
- net 5V: now also Q1.3 (D)
- net GND: now also U1.1 (GND)
- net at C2.1, D1.1 (K), R2.1: now also Q1.1 (G)
- net at D2.2 (A), R3.1: now also Q1.2 (S)
- net at C3.2, D2.1 (K): now also U1.3 (VI)
Changed lines of the file:
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@@
     (pin "2")
-  )
-  (symbol (lib_id "Device:Q_PMOS_GSD") (at 140.335 36.195 270) (mirror x) (unit 1)
-    (in_bom yes) (on_board yes) (fields_autoplaced)
-    (property "Reference" "Q1" (id 0) (at 140.335 26.035 90))
-    (property "Value" "IRF7425" (id 1) (at 140.335 28.575 90))
-    (property "Footprint" "Package_SO:SO-8_3.9x4.9mm_P1.27mm" (id 2) (at 142.875 31.115 0)
-      (effects (font (size 1.27 1.27)) hide)
-    )
-    (property "Datasheet" "~" (id 3) (at 140.335 36.195 0)
-      (effects (font (size 1.27 1.27)) hide)
-    )
-    (pin "1")
-    (pin "2")
-    (pin "3")
   )
   (symbol (lib_id "Device:D_Schottky") (at 164.465 33.655 180) (unit 1)
     (in_bom yes) (on_board yes) (fields_autoplaced)
     (property "Reference" "D2" (id 0) (at 164.7825 26.67 0))
-    (property "Value" "1N5822" (id 1) (at 164.7825 29.21 0))
+    (property "Value" "SS210" (id 1) (at 164.7825 29.21 0))
     (property "Footprint" "" (id 2) (at 164.465 33.655 0)
       (effects (font (size 1.27 1.27)) hide)
@@
     (pin "2")
   )
+  (symbol (lib_id "Transistor_FET:AO3401A") (at 140.335 36.195 90) (unit 1)
+    (in_bom yes) (on_board yes) (fields_autoplaced)
+    (property "Reference" "Q1" (id 0) (at 140.335 26.035 90))
+    (property "Value" "AO3401A" (id 1) (at 140.335 28.575 90))
+    (property "Footprint" "Package_TO_SOT_SMD:SOT-23" (id 2) (at 142.24 31.115 0)
+      (effects (font (size 1.27 1.27) italic) (justify left) hide)
+    )
+    (property "Datasheet" "http://www.aosmd.com/pdfs/datasheet/AO3401A.pdf" (id 3) (at 140.335 36.195 0)
+      (effects (font (size 1.27 1.27)) (justify left) hide)
+    )
+    (pin "1")
+    (pin "2")
+    (pin "3")
+  )
   (symbol (lib_id "power:GND") (at 116.205 64.135 0) (unit 1)
     (in_bom yes) (on_board yes) (fields_autoplaced)
@@
     (pin "2")
   )
-  (symbol (lib_id "Regulator_Linear:LD1117S33TR_SOT223") (at 191.77 33.655 0) (unit 1)
-    (in_bom yes) (on_board yes) (fields_autoplaced)
-    (property "Reference" "U1" (id 0) (at 191.77 26.035 0))
-    (property "Value" "LD1117S33TR_SOT223" (id 1) (at 191.77 28.575 0))
-    (property "Footprint" "Package_TO_SOT_SMD:SOT-223-3_TabPin2" (id 2) (at 191.77 28.575 0)
-      (effects (font (size 1.27 1.27)) hide)
-    )
-    (property "Datasheet" "http://www.st.com/st-web-ui/static/active/en/resource/technical/document/datasheet/CD00000544.pdf" (id 3) (at 194.31 40.005 0)
+  (symbol (lib_id "Regulator_Linear:LM1117-3.3") (at 191.77 33.655 0) (unit 1)
+    (in_bom yes) (on_board yes) (fields_autoplaced)
+    (property "Reference" "U1" (id 0) (at 191.77 26.67 0))
+    (property "Value" "LM1117-3.3" (id 1) (at 191.77 29.21 0))
+    (property "Footprint" "" (id 2) (at 191.77 33.655 0)
+      (effects (font (size 1.27 1.27)) hide)
+    )
+    (property "Datasheet" "http://www.ti.com/lit/ds/symlink/lm1117.pdf" (id 3) (at 191.77 33.655 0)
       (effects (font (size 1.27 1.27)) hide)
     )
@@
     (in_bom yes) (on_board yes) (fields_autoplaced)
     (property "Reference" "D1" (id 0) (at 132.3975 42.545 0))
-    (property "Value" "1N5822" (id 1) (at 132.3975 45.085 0))
+    (property "Value" "SS210" (id 1) (at 132.3975 45.085 0))
     (property "Footprint" "" (id 2) (at 132.08 49.53 0)
       (effects (font (size 1.27 1.27)) hide)
@@
     )
     (path "/f08cf256-66f8-440b-9c81-3b565d9bbcdf"
-      (reference "D1") (unit 1) (value "1N5822") (footprint "")
+      (reference "D1") (unit 1) (value "SS210") (footprint "")
     )
     (path "/3e872b0a-69c3-4a00-850a-b1339cea7290"
-      (reference "D2") (unit 1) (value "1N5822") (footprint "")
+      (reference "D2") (unit 1) (value "SS210") (footprint "")
     )
     (path "/5c36d873-bd20-4df5-9fe7-2f8ba335a3e3"
@@
       (reference "J2") (unit 1) (value "Vout") (footprint "TerminalBlock:TerminalBlock_bornier-2_P5.08mm")
     )
-    (path "/1374b80f-d43b-4c6d-a8d5-e4cb24f3116a"
-      (reference "Q1") (unit 1) (value "IRF7425") (footprint "Package_SO:SO-8_3.9x4.9mm_P1.27mm")
+    (path "/88e3e48d-edc7-4566-877b-292a06d60e45"
+      (reference "Q1") (unit 1) (value "AO3401A") (footprint "Package_TO_SOT_SMD:SOT-23")
     )
     (path "/04517978-c793-4358-8777-4549188e483e"
@@
       (reference "R3") (unit 1) (value "100") (footprint "")
     )
-    (path "/c60e1097-081c-47c0-b01b-4ea2df6b0304"
-      (reference "U1") (unit 1) (value "LD1117S33TR_SOT223") (footprint "Package_TO_SOT_SMD:SOT-223-3_TabPin2")
-    )
-  )
+    (path "/c6bef878-217a-4fca-bcd3-afcb5883b6cf"
+      (reference "U1") (unit 1) (value "LM1117-3.3") (footprint "")
+    )
+  )
